File: hardware/schematics/kicad/main.kicad_sch (KiCad schematic)
At the start: 301 parts, among them IC1 74257N, IC10 74181N, IC100 74257N, IC101 74377N, IC102 74377N, IC103 74153N, IC104 74257N, IC105 74148N, IC106 74377N, IC107 7474N, IC108 7474N, IC109 74377N, IC11 74181N, IC110 74377N, IC111 74253N, IC112 74257N, IC113 74253N, IC114 74257N, IC115 7404N, IC116 74153N, IC117 74377N, IC118 74257N, IC119 7408N, IC12 74151N, IC120 74244N, IC121 74257N, IC122 74257N, IC123 74377N, IC124 74153N, IC125 74257N, IC126 7474N, IC127 74257N, IC128 74157N, IC129 74157N, IC13 74257N, IC130 74151N, IC131 74157N, IC132 74157N, IC133 74151N, IC134 74273N, IC135 74273N, IC136 74273N, IC137 7474N, IC138 7404N, IC139 7400N, IC14 74151N, IC140 58C256P, IC141 74151N, IC142 74257N, IC143 7408N, IC144 74151N, IC145 7410N, IC146 7408N, IC147 74257N, IC148 7400N, IC149 74138N, IC15 74257N, IC150 74244N, IC151 7432N, IC152 74151N, IC153 7432N, IC154 7404N, IC155 7404N, IC156 7404N, IC157 74377N, IC158 74377N, IC159 74377N, IC16 74151N, IC160 74151N, IC161 74244N, IC162 74377N, IC163 74244N, IC164 74138N, IC165 74377N, IC166 74377N, IC167 7432N, IC168 7420N, IC169 74377N, IC17 74244N, IC170 74253N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

Commit message: kicad
Connections:
- net GND: now also IC130.7 (G), IC133.7 (G), IC141.7 (G), IC144.7 (G), IC152.7 (G), IC160.7 (G), IC2.7 (G), IC20.7 (G), IC3.7 (G), IC30.7 (G), IC41.7 (G), IC42.7 (G), IC44.7 (G), IC5.7 (G), IC53.7 (G), IC56.7 (G), IC6.7 (G), IC62.7 (G), IC67.7 (G), IC68.7 (G), IC69.7 (G), IC71.7 (G), IC80.7 (G), IC81.7 (G), IC82.7 (G), IC84.7 (G), IC85.7 (G), IC86.7 (G), IC87.7 (G), IC88.7 (G), IC89.7 (G), IC9.7 (G)
- net alu_a_src_0_muxed: now also IC130.11 (A), IC133.11 (A), IC141.11 (A), IC144.11 (A), IC152.11 (A), IC160.11 (A), IC2.11 (A), IC20.11 (A), IC3.11 (A), IC30.11 (A), IC41.11 (A), IC44.11 (A), IC5.11 (A), IC53.11 (A), IC56.11 (A), IC6.11 (A), IC62.11 (A), IC67.11 (A), IC68.11 (A), IC69.11 (A), IC71.11 (A), IC80.11 (A), IC81.11 (A), IC82.11 (A), IC84.11 (A), IC85.11 (A), IC86.11 (A), IC87.11 (A), IC88.11 (A), IC89.11 (A), IC9.11 (A)
- net alu_a_src_1_muxed: now also IC130.10 (B), IC133.10 (B), IC141.10 (B), IC144.10 (B), IC152.10 (B), IC160.10 (B), IC2.10 (B), IC20.10 (B), IC3.10 (B), IC30.10 (B), IC41.10 (B), IC44.10 (B), IC5.10 (B), IC53.10 (B), IC56.10 (B), IC6.10 (B), IC62.10 (B), IC67.10 (B), IC68.10 (B), IC69.10 (B), IC71.10 (B), IC80.10 (B), IC81.10 (B), IC82.10 (B), IC84.10 (B), IC85.10 (B), IC86.10 (B), IC87.10 (B), IC88.10 (B), IC89.10 (B), IC9.10 (B)
- net alu_a_src_2_muxed: now also IC130.9 (C), IC133.9 (C), IC141.9 (C), IC144.9 (C), IC152.9 (C), IC160.9 (C), IC2.9 (C), IC20.9 (C), IC3.9 (C), IC30.9 (C), IC41.9 (C), IC44.9 (C), IC5.9 (C), IC53.9 (C), IC56.9 (C), IC6.9 (C), IC62.9 (C), IC67.9 (C), IC68.9 (C), IC69.9 (C), IC71.9 (C), IC80.9 (C), IC81.9 (C), IC82.9 (C), IC84.9 (C), IC85.9 (C), IC86.9 (C), IC87.9 (C), IC88.9 (C), IC89.9 (C), IC9.9 (C)

Commit message: kicad
Connections:
- net mdr_0_wrt is gone; now on net clk: IC19.1 (G)
- net GND: now also IC1.15 (G), IC103.1 (1G), IC103.15 (2G), IC111.1 (1G), IC111.15 (2G), IC113.1 (1G), IC113.15 (2G), IC116.1 (1G), IC116.15 (2G), IC12.12 (D7), IC12.13 (D6), IC124.1 (1G), IC124.15 (2G), IC128.15 (G), IC129.15 (G), IC13.15 (G), IC130.12 (D7), IC130.13 (D6), IC130.14 (D5), IC131.15 (G), IC132.15 (G), IC133.12 (D7), IC133.13 (D6), IC133.14 (D5), IC14.7 (G), IC141.12 (D7), IC141.13 (D6), IC141.14 (D5), IC142.15 (G), IC144.12 (D7), IC144.13 (D6), IC144.14 (D5), IC147.15 (G), IC152.12 (D7), IC152.13 (D6), IC152.14 (D5), IC160.12 (D7), IC160.13 (D6), IC160.14 (D5), IC180.1 (1G), IC180.15 (2G), IC23.7 (G), IC24.15 (G), IC241.1 (1G), IC241.10 (2C0), IC241.11 (2C1), IC241.12 (2C2), IC241.13 (2C3), IC241.15 (2G), IC255.1 (1G), IC255.15 (2G), IC29.1 (1G), IC29.15 (2G), IC341.10 (3B), IC341.11 (3A), IC341.13 (4B), IC341.14 (4A), IC341.15 (G), IC341.5 (2A), IC341.6 (2B), IC42.12 (D7), IC42.13 (D6), IC42.14 (D5), IC64.1 (1G), IC64.15 (2G), IC7.15 (G), IC80.12 (D7), IC80.13 (D6), IC80.14 (D5), IC83.1 (1G), IC83.15 (2G), IC91.1 (1G), IC91.15 (2G), IC92.1 (1G), IC92.15 (2G), IC95.1 (1G), IC95.15 (2G)
- net alu_b_src_0: now also IC103.14 (A), IC116.14 (A), IC124.14 (A)
- net alu_b_src_1: now also IC103.2 (B), IC116.2 (B), IC124.2 (B)
- net clk: now also FLAGS0.11 (CLK), IC101.11 (CLK), IC102.11 (CLK), IC106.11 (CLK), IC109.11 (CLK), IC110.11 (CLK), IC117.11 (CLK), IC123.11 (CLK), IC157.11 (CLK), IC158.11 (CLK), IC159.11 (CLK), IC162.11 (CLK), IC165.11 (CLK), IC166.11 (CLK), IC169.11 (CLK), IC171.11 (CLK), IC172.11 (CLK), IC177.11 (CLK), IC178.11 (CLK), IC183.11 (CLK), IC183.13 (5D), IC183.14 (6D), IC183.17 (7D), IC183.18 (8D), IC183.3 (1D), IC183.4 (2D), IC183.7 (3D), IC183.8 (4D), IC184.11 (CLK), IC19.11 (CLK), IC19.13 (5D), IC19.14 (6D), IC19.17 (7D), IC19.18 (8D), IC19.3 (1D), IC19.4 (2D), IC19.7 (3D), IC19.8 (4D), IC198.11 (CLK), IC204.11 (CLK), IC210.11 (CLK), IC231.11 (CLK), IC24.12 (4Y), IC24.4 (1Y), IC24.7 (2Y), IC24.9 (3Y), IC245.11 (CLK), IC260.11 (CLK), IC31.11 (CLK), IC48.11 (CLK), IC57.11 (CLK), IC66.11 (CLK), IC7.12 (4Y), IC7.4 (1Y), IC7.7 (2Y), IC7.9 (3Y), INT_CODE_REG1.11 (CLK), INT_STATUS_REG0.11 (CLK)
- net data_bus0: now also U1.13 (DQ0)
- net data_bus1: now also U1.14 (DQ1)
- net data_bus2: now also U1.15 (DQ2)
- net data_bus3: now also U1.17 (DQ3)
- net data_bus4: now also U1.18 (DQ4)
- net data_bus5: now also U1.19 (DQ5)
- net data_bus6: now also U1.20 (DQ6)
- net data_bus7: now also U1.21 (DQ7)
- net gh_wrt: now also IC204.1 (G)
- net gl_wrt: now also IC184.1 (G)
- net ~{clear_all_ints}: now also IC143.10 (I1), IC143.12 (I0), IC143.5 (I1), IC146.1 (I0), IC146.12 (I0), IC146.4 (I0), IC146.9 (I0), IC149.10 (Y5), IC149.11 (Y4), IC149.12 (Y3), IC149.13 (Y2), IC149.14 (Y1), IC149.7 (Y7), IC149.9 (Y6)
- no-connect marks 57 -> 75
Other:
- moved on the sheet: FLAGS0A, IC100A, IC101A, IC102A, IC103A, IC104A, IC105A, IC106A, IC107A, IC107B, IC108A, IC108B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

Commit message: kicad
Parts:
- removed IC150: 74244N, main:DIL20, symbol main-eagle-import:74xx-eu_74244N
- removed IC151: 7432N, main:DIL14, symbol main-eagle-import:7432N
- removed IC154, IC155, IC156: 7404N, main:DIL14, symbol main-eagle-import:7404N
- added IC150, IC70: 7404N, main:DIL14, symbol main-eagle-import:7404N
- added IC154: 74244N, main:DIL20, symbol main-eagle-import:74xx-eu_74244N
Connections:
- net alu_op0 is gone; now on net alu_op_0: IC10.6 (S0), IC11.6 (S0), IC_10_0.1 (I0)
- net alu_op1 is gone; now on net alu_op_1: IC10.5 (S1), IC11.5 (S1), IC_02_0.3 (I1)
- net alu_op2 is gone; now on net alu_op_2: IC10.4 (S2), IC11.4 (S2), IC_02_0.2 (I0)
- net alu_op3 is gone; now on net alu_op_3: IC10.3 (S3), IC11.3 (S3), IC_10_0.2 (I1)
- net clear_all_ints is gone; now on net clear_all_irqs: IC196.3 (I)
- net mdr_1_wrt is gone; now on net mdrh_wrt: IC183.1 (G)
- net mdr_data_out is gone; now on net mdr_out_en: IC43.5 (I)
- net msw_h_wrt is gone; now on net upper_flags_wrt: IC206.1 (~{A}/B)
- net ssph0 is gone; now on net ksph0: IC42.3 (D1)
- net sspl0 is gone; now on net kspl0: IC42.4 (D0)
- net status_flags_wrt is gone; now on net status_wrt: IC259.19 (Q8)
- net tdrh_0 is gone; now on net tdrh0: IC9.12 (D7), IC92.3 (1C3)
- net tdrh_1 is gone; now on net tdrh1: IC5.12 (D7), IC92.13 (2C3)
- net tdrh_2 is gone; now on net tdrh2: IC103.3 (1C3), IC30.12 (D7)
- net tdrh_3 is gone; now on net tdrh3: IC103.13 (2C3), IC53.12 (D7)
- net tdrh_4 is gone; now on net tdrh4: IC116.3 (1C3), IC67.12 (D7)
- net tdrh_5 is gone; now on net tdrh5: IC116.13 (2C3), IC71.12 (D7)
- net tdrh_6 is gone; now on net tdrh6: IC124.3 (1C3), IC84.12 (D7)
- net tdrh_7 is gone; now on net tdrh7: IC124.13 (2C3), IC87.12 (D7)
- net tdrl_0 is gone; now on net tdrl0: IC9.13 (D6), IC92.4 (1C2)
- net tdrl_1 is gone; now on net tdrl1: IC5.13 (D6), IC92.12 (2C2)
- net tdrl_2 is gone; now on net tdrl2: IC103.4 (1C2), IC30.13 (D6)
- net tdrl_3 is gone; now on net tdrl3: IC103.12 (2C2), IC53.13 (D6)
- net tdrl_4 is gone; now on net tdrl4: IC116.4 (1C2), IC67.13 (D6)
- net tdrl_5 is gone; now on net tdrl5: IC116.12 (2C2), IC71.13 (D6)
- net tdrl_6 is gone; now on net tdrl6: IC124.4 (1C2), IC84.13 (D6)
- net tdrl_7 is gone; now on net tdrl7: IC124.12 (2C2), IC87.13 (D6)
- net zbus_4 is gone; now on net zbus4: IC206.3 (1B)
- net zbus_5 is gone; now on net zbus5: IC206.6 (2B)
- net zbus_6 is gone; now on net zbus6: IC206.10 (3B)
- net zbus_7 is gone; now on net zbus7: IC206.13 (4B)
- net zbus_src_0 is gone; now on net zbus_in_src_0: IC111.14 (A), IC113.14 (A), IC91.14 (A), IC95.14 (A)
- net zbus_src_1 is gone; now on net zbus_in_src_1: IC111.2 (B), IC113.2 (B), IC91.2 (B), IC95.2 (B)
- net GND: now also IC229.6 (A3), IC229.8 (A4), IC230.2 (A1), IC230.4 (A2), IC230.6 (A3), IC230.8 (A4), IC27.8 (A4), IC72.4 (A2), IC72.6 (A3), IC72.8 (A4), IC154.6 (A3), IC154.8 (A4)
- net alu_a_src_3: no longer IC83.14 (A)
- net alu_a_src_3_muxed: now also IC29.14 (A), IC64.14 (A), IC83.14 (A)
- net alu_a_src_4: no longer IC83.2 (B)
- net alu_a_src_4_muxed: now also IC29.2 (B), IC64.2 (B), IC83.2 (B)
- net bus_rd: now also IC154.18 (Y1)
- net bus_tristate: now also IC154.1 (G)
- net bus_wr: now also IC154.16 (Y2)
- net clk: no longer IC183.13 (5D), IC183.14 (6D), IC183.17 (7D), IC183.18 (8D), IC183.3 (1D), IC183.4 (2D), IC183.7 (3D), IC183.8 (4D), IC19.1 (G), IC19.13 (5D), IC19.14 (6D), IC19.17 (7D), IC19.18 (8D), IC19.3 (1D), IC19.4 (2D), IC19.7 (3D), IC19.8 (4D), IC24.12 (4Y), IC24.4 (1Y), IC24.7 (2Y), IC24.9 (3Y), IC7.12 (4Y), IC7.4 (1Y), IC7.7 (2Y), IC7.9 (3Y)
- net data_bus0: no longer IC24.14 (4A)
- net mdr_out_src: now also IC54.1 (~{A}/B), IC96.1 (~{A}/B)
- net mdrl_wrt: now also IC19.1 (G)
- net rd: now also IC70.9 (I)
- net wr: now also IC150.9 (I)
- net zbus0: now also IC184.3 (1D), IC204.3 (1D), IC7.2 (1A), IC99.3 (1D)
- net zbus1: now also IC184.4 (2D), IC204.4 (2D), IC7.5 (2A), IC99.4 (2D)
- net zbus2: now also IC184.7 (3D), IC204.7 (3D), IC7.11 (3A), IC99.7 (3D)
- net zbus3: now also IC184.8 (4D), IC204.8 (4D), IC7.14 (4A), IC99.8 (4D)
- net zbus4: now also IC184.13 (5D), IC204.13 (5D), IC24.2 (1A), IC99.13 (5D)
- net zbus5: now also IC184.14 (6D), IC204.14 (6D), IC24.5 (2A), IC99.14 (6D)
- net zbus6: now also IC184.17 (7D), IC204.17 (7D), IC24.11 (3A), IC99.17 (7D)
- net zbus7: now also IC184.18 (8D), IC204.18 (8D), IC24.14 (4A), IC99.18 (8D)
- net tdrl4: now reaches IC157.12 (5Q)
- net tdrl5: now reaches IC157.15 (6Q)
- net tdrl6: now reaches IC157.16 (7Q)
- net tdrl7: now reaches IC157.19 (8Q)
- net tdrl0: now reaches IC157.2 (1Q)
- net tdrl1: now reaches IC157.5 (2Q)
- net tdrl2: now reaches IC157.6 (3Q)
- net tdrl3: now reaches IC157.9 (4Q)
- net tdrh4: now reaches IC158.12 (5Q)
- net tdrh5: now reaches IC158.15 (6Q)
- net tdrh6: now reaches IC158.16 (7Q)
- net tdrh7: now reaches IC158.19 (8Q)
- net tdrh0: now reaches IC158.2 (1Q)
- net tdrh1: now reaches IC158.5 (2Q)
- net tdrh2: now reaches IC158.6 (3Q)
- net tdrh3: now reaches IC158.9 (4Q)
- net upper_flags_wrt: now reaches IC79.2 (Q1)
- net mdr_0_1 renamed mdrl_1
- net mdr_0_2 renamed mdrl_2
- net mdr_0_3 renamed mdrl_3
- removed net mdr_0_4: IC116.10 (2C0), IC116.11 (2C1), IC116.5 (1C1), IC116.6 (1C0), IC124.10 (2C0), IC124.11 (2C1), IC124.5 (1C1), IC124.6 (1C0), IC183.12 (5Q), IC183.15 (6Q), IC183.16 (7Q), IC183.19 (8Q), IC185.11 (A1), IC185.13 (A2), IC185.15 (A3), IC185.17 (A4), IC19.12 (5Q), IC19.15 (6Q), IC19.16 (7Q), IC19.19 (8Q), IC43.6 (O), IC54.1 (~{A}/B), IC54.15 (G), IC67.14 (D5), IC67.15 (D4), IC71.14 (D5), IC71.15 (D4), IC84.14 (D5), IC84.15 (D4), IC87.14 (D5), IC87.15 (D4), IC96.1 (~{A}/B), IC96.10 (3B), IC96.11 (3A), IC96.13 (4B), IC96.14 (4A), IC96.15 (G), IC96.2 (1A), IC96.3 (1B), IC96.5 (2A), IC96.6 (2B), IC97.11 (A1), IC97.13 (A2), IC97.15 (A3), IC97.17 (A4)
- net mdr_1_1 renamed mdrh_1
- net mdr_1_2 renamed mdrh_2
- net mdr_1_3 renamed mdrh_3
- net msw_12 renamed flags_4
- net msw_13 renamed flags_5
- net msw_14 renamed flags_6
- net flags_6: no longer IC182.5 (1C1), IC99.16 (7Q)
- net msw_15 renamed flags_7
- net msw_cf renamed flags_cf
- net msw_cpu_mode renamed status_cpu_mode
- net msw_dir renamed status_dir
- net msw_display_reg_load renamed status_display_reg_load
- net msw_dma_ack renamed status_dma_ack
- net msw_halt renamed status_halt
- net msw_interrupt_enable renamed status_irq_enable
- net msw_l_wrt renamed status_wrt
- net msw_of renamed flags_of
- net msw_paging_en renamed status_paging_en
- net msw_sf renamed flags_sf
- net msw_zf renamed flags_zf
- removed net ~{clear_all_ints}: IC143.1 (I0), IC143.10 (I1), IC143.12 (I0), IC143.13 (I1), IC143.4 (I0), IC143.5 (I1), IC143.9 (I0), IC146.1 (I0), IC146.10 (I1), IC146.12 (I0), IC146.13 (I1), IC146.2 (I1), IC146.4 (I0), IC146.5 (I1), IC146.9 (I0), IC149.10 (Y5), IC149.11 (Y4), IC149.12 (Y3), IC149.13 (Y2), IC149.14 (Y1), IC149.7 (Y7), IC149.9 (Y6), IC196.4 (O)
- new net: IC146.9 (I0), IC149.9 (Y6)
- new net: IC146.1 (I0), IC149.11 (Y4)
- new net: IC183.13 (5D), IC19.13 (5D), IC24.4 (1Y)
- new net: IC183.14 (6D), IC19.14 (6D), IC24.7 (2Y)
- new net: IC183.17 (7D), IC19.17 (7D), IC24.9 (3Y)
- new net: IC183.18 (8D), IC19.18 (8D), IC24.12 (4Y)
- new net: IC183.3 (1D), IC19.3 (1D), IC7.4 (1Y)
- new net: IC183.4 (2D), IC19.4 (2D), IC7.7 (2Y)
- new net: IC183.7 (3D), IC19.7 (3D), IC7.9 (3Y)
- new net: IC183.8 (4D), IC19.8 (4D), IC7.12 (4Y)
- new net: IC143.5 (I1), IC149.14 (Y1)
- new net: IC146.4 (I0), IC149.10 (Y5)
- new net: IC43.6 (O), IC54.15 (G), IC96.15 (G)
- new net: IC154.2 (A1), IC70.8 (O)
- new net: IC146.12 (I0), IC149.7 (Y7)
- new net: IC143.12 (I0), IC149.12 (Y3)
- new net: IC143.10 (I1), IC149.13 (Y2)
- new net: IC150.8 (O), IC154.4 (A2)
- new net mdrh_4: IC116.5 (1C1), IC183.12 (5Q), IC185.11 (A1), IC67.14 (D5), IC96.3 (1B)
- new net mdrh_5: IC116.11 (2C1), IC183.15 (6Q), IC185.13 (A2), IC71.14 (D5), IC96.6 (2B)
- new net mdrh_6: IC124.5 (1C1), IC183.16 (7Q), IC185.15 (A3), IC84.14 (D5), IC96.10 (3B)
- new net mdrh_7: IC124.11 (2C1), IC183.19 (8Q), IC185.17 (A4), IC87.14 (D5), IC96.13 (4B)
- new net mdrl_4: IC116.6 (1C0), IC19.12 (5Q), IC67.15 (D4), IC96.2 (1A), IC97.11 (A1)
- new net mdrl_5: IC116.10 (2C0), IC19.15 (6Q), IC71.15 (D4), IC96.5 (2A), IC97.13 (A2)
- new net mdrl_6: IC124.6 (1C0), IC19.16 (7Q), IC84.15 (D4), IC96.11 (3A), IC97.15 (A3)
- new net mdrl_7: IC124.10 (2C0), IC19.19 (8Q), IC87.15 (D4), IC96.14 (4A), IC97.17 (A4)
- new net status_6: IC182.5 (1C1), IC99.16 (7Q)
- new net ~{clear_all_irqs}: IC143.1 (I0), IC143.13 (I1), IC143.4 (I0), IC143.9 (I0), IC146.10 (I1), IC146.13 (I1), IC146.2 (I1), IC146.5 (I1), IC196.4 (O)
- no-connect marks 75 -> 132
Other:
- note added: "flags"
- note removed: "msw_h"
- moved on the sheet: IC43C, IC99A

Commit message: kicad
Connections:
- net vss is gone; now on net GND: IC140.14 (VSS), IC21.14 (VSS)
- net address_bus0: now also U1.12 (A0), U2.12 (A0), U3.12 (A0), U4.12 (A0), U5.12 (A0), U6.12 (A0), U7.12 (A0), U8.12 (A0)
- net address_bus1: now also U1.11 (A1), U2.11 (A1), U3.11 (A1), U4.11 (A1), U5.11 (A1), U6.11 (A1), U7.11 (A1), U8.11 (A1)
- net address_bus10: now also U1.23 (A10), U2.23 (A10), U3.23 (A10), U4.23 (A10), U5.23 (A10), U6.23 (A10), U7.23 (A10), U8.23 (A10)
- net address_bus11: now also U1.25 (A11), U2.25 (A11), U3.25 (A11), U4.25 (A11), U5.25 (A11), U6.25 (A11), U7.25 (A11), U8.25 (A11)
- net address_bus12: now also U1.4 (A12), U2.4 (A12), U3.4 (A12), U4.4 (A12), U5.4 (A12), U6.4 (A12), U7.4 (A12), U8.4 (A12)
- net address_bus13: now also U1.28 (A13), U2.28 (A13), U3.28 (A13), U4.28 (A13), U5.28 (A13), U6.28 (A13), U7.28 (A13), U8.28 (A13)
- net address_bus14: now also U1.3 (A14), U2.3 (A14), U3.3 (A14), U4.3 (A14), U5.3 (A14), U6.3 (A14), U7.3 (A14), U8.3 (A14)
- net address_bus15: now also U1.31 (A15), U2.31 (A15), U3.31 (A15), U4.31 (A15), U5.31 (A15), U6.31 (A15), U7.31 (A15), U8.31 (A15)
- net address_bus16: now also U1.2 (A16), U2.2 (A16), U3.2 (A16), U4.2 (A16), U5.2 (A16), U6.2 (A16), U7.2 (A16), U8.2 (A16)
- net address_bus17: now also U1.30 (A17), U2.30 (A17), U3.30 (A17), U4.30 (A17), U5.30 (A17), U6.30 (A17), U7.30 (A17), U8.30 (A17)
- net address_bus18: now also U1.1 (A18), U2.1 (A18), U3.1 (A18), U4.1 (A18), U5.1 (A18), U6.1 (A18), U7.1 (A18), U8.1 (A18)
- net address_bus2: now also U1.10 (A2), U2.10 (A2), U3.10 (A2), U4.10 (A2), U5.10 (A2), U6.10 (A2), U7.10 (A2), U8.10 (A2)
- net address_bus3: now also U1.9 (A3), U2.9 (A3), U3.9 (A3), U4.9 (A3), U5.9 (A3), U6.9 (A3), U7.9 (A3), U8.9 (A3)
- net address_bus4: now also U1.8 (A4), U2.8 (A4), U3.8 (A4), U4.8 (A4), U5.8 (A4), U6.8 (A4), U7.8 (A4), U8.8 (A4)
- net address_bus5: now also U1.7 (A5), U2.7 (A5), U3.7 (A5), U4.7 (A5), U5.7 (A5), U6.7 (A5), U7.7 (A5), U8.7 (A5)
- net address_bus6: now also U1.6 (A6), U2.6 (A6), U3.6 (A6), U4.6 (A6), U5.6 (A6), U6.6 (A6), U7.6 (A6), U8.6 (A6)
- net address_bus7: now also U1.5 (A7), U2.5 (A7), U3.5 (A7), U4.5 (A7), U5.5 (A7), U6.5 (A7), U7.5 (A7), U8.5 (A7)
- net address_bus8: now also U1.27 (A8), U2.27 (A8), U3.27 (A8), U4.27 (A8), U5.27 (A8), U6.27 (A8), U7.27 (A8), U8.27 (A8)
- net address_bus9: now also U1.26 (A9), U2.26 (A9), U3.26 (A9), U4.26 (A9), U5.26 (A9), U6.26 (A9), U7.26 (A9), U8.26 (A9)
- net data_bus0: now also U2.13 (DQ0), U3.13 (DQ0), U4.13 (DQ0), U5.13 (DQ0), U6.13 (DQ0), U7.13 (DQ0), U8.13 (DQ0)
- net data_bus1: now also U2.14 (DQ1), U3.14 (DQ1), U4.14 (DQ1), U5.14 (DQ1), U6.14 (DQ1), U7.14 (DQ1), U8.14 (DQ1)
- net data_bus2: now also U2.15 (DQ2), U3.15 (DQ2), U4.15 (DQ2), U5.15 (DQ2), U6.15 (DQ2), U7.15 (DQ2), U8.15 (DQ2)
- net data_bus3: now also U2.17 (DQ3), U3.17 (DQ3), U4.17 (DQ3), U5.17 (DQ3), U6.17 (DQ3), U7.17 (DQ3), U8.17 (DQ3)
- net data_bus4: now also U2.18 (DQ4), U3.18 (DQ4), U4.18 (DQ4), U5.18 (DQ4), U6.18 (DQ4), U7.18 (DQ4), U8.18 (DQ4)
- net data_bus5: now also U2.19 (DQ5), U3.19 (DQ5), U4.19 (DQ5), U5.19 (DQ5), U6.19 (DQ5), U7.19 (DQ5), U8.19 (DQ5)
- net data_bus6: now also U2.20 (DQ6), U3.20 (DQ6), U4.20 (DQ6), U5.20 (DQ6), U6.20 (DQ6), U7.20 (DQ6), U8.20 (DQ6)
- net data_bus7: now also U2.21 (DQ7), U3.21 (DQ7), U4.21 (DQ7), U5.21 (DQ7), U6.21 (DQ7), U7.21 (DQ7), U8.21 (DQ7)
Other:
- note added: "These 3 signals are used in the memory decoder and hence show as dangling here."

Commit message: kicad
Parts:
- added R29, R30, R31, R32, R33, R34, R35, R36, R37, R38, R39, R40, R41, R42, R43, R44, R45, R46, R47, R48, R49, R50, R51, R52, R53, R54, R55, R56, R57, R58, R59, R60: R-US_0204/2V, main:0204V, symbol main-eagle-import:R-US_0204/2V
- added SW6, SW7, SW8, SW9: SW_DIP-8, main:EDG-08, symbol main-eagle-import:SW_DIP-8
Connections:
- net ~{bus_tristate} is gone; now on net GND: IC176.8 (O), IC218.1 (G), IC219.1 (G), IC222.1 (G), IC223.1 (G), IC224.1 (G), IC225.1 (G), IC228.1 (G), IC229.1 (G), IC230.1 (G), IC27.1 (G)
- net GND: now also SW6.10, SW6.11, SW6.12, SW6.13, SW6.14, SW6.15, SW6.16, SW6.9, SW7.10, SW7.11, SW7.12, SW7.13, SW7.14, SW7.15, SW7.16, SW7.9, SW8.10, SW8.11, SW8.12, SW8.13, SW8.14, SW8.15, SW8.16, SW8.9, SW9.10, SW9.11, SW9.12, SW9.13, SW9.14, SW9.15, SW9.16, SW9.9
- net VCC: now also R29.2, R30.2, R31.2, R32.2, R33.2, R34.2, R35.2, R36.2, R37.2, R38.2, R39.2, R40.2, R41.2, R42.2, R43.2, R44.2, R45.2, R46.2, R47.2, R48.2, R49.2, R50.2, R51.2, R52.2, R53.2, R54.2, R55.2, R56.2, R57.2, R58.2, R59.2, R60.2
- net panel_address_0: now also R29.1, SW6.8
- net panel_address_1: now also R30.1, SW6.7
- net panel_address_10: now also R39.1, SW7.6
- net panel_address_11: now also R40.1, SW7.5
- net panel_address_12: now also R41.1, SW7.4
- net panel_address_13: now also R42.1, SW7.3
- net panel_address_14: now also R43.1, SW7.2
- net panel_address_15: now also R44.1, SW7.1
- net panel_address_16: now also R45.1, SW8.8
- net panel_address_17: now also R46.1, SW8.7
- net panel_address_18: now also R47.1, SW8.6
- net panel_address_19: now also R48.1, SW8.5
- net panel_address_2: now also R31.1, SW6.6
- net panel_address_20: now also R49.1, SW8.4
- net panel_address_21: now also R50.1, SW8.3
- net panel_address_3: now also R32.1, SW6.5
- net panel_address_4: now also R33.1, SW6.4
- net panel_address_5: now also R34.1, SW6.3
- net panel_address_6: now also R35.1, SW6.2
- net panel_address_7: now also R36.1, SW6.1
- net panel_address_8: now also R37.1, SW7.8
- net panel_address_9: now also R38.1, SW7.7
- net panel_data_0: now also R53.1, SW9.8
- net panel_data_1: now also R54.1, SW9.7
- net panel_data_2: now also R55.1, SW9.6
- net panel_data_3: now also R56.1, SW9.5
- net panel_data_4: now also R57.1, SW9.4
- net panel_data_5: now also R58.1, SW9.3
- net panel_data_6: now also R59.1, SW9.2
- net panel_data_7: now also R60.1, SW9.1
- new net: R52.1, SW8.1
- new net: R51.1, SW8.2
Other:
- moved on the sheet: IC218A, IC219A, IC222A, IC223A, IC224A, IC225A, IC228A, IC229A, IC230A
