File: hardware/schematics/kicad/main.kicad_sch (KiCad schematic)
At the start: 335 parts, among them IC1 74257N, IC10 74181N, IC100 74257N, IC101 74377N, IC102 74377N, IC103 74153N, IC104 74257N, IC105 74148N, IC106 74377N, IC107 7474N, IC108 7474N, IC109 74377N, IC11 74181N, IC110 74377N, IC111 74253N, IC112 74257N, IC113 74253N, IC114 74257N, IC115 7404N, IC116 74153N, IC117 74377N, IC118 74257N, IC119 7408N, IC12 74151N, IC120 74244N, IC121 74257N, IC122 74257N, IC123 74377N, IC124 74153N, IC125 74257N, IC126 7474N, IC127 74257N, IC128 74157N, IC129 74157N, IC13 74257N, IC130 74151N, IC131 74157N, IC132 74157N, IC133 74151N, IC134 74273N, IC135 74273N, IC136 74273N, IC137 7474N, IC138 7404N, IC139 7400N, IC14 74151N, IC140 58C256P, IC141 74151N, IC142 74257N, IC143 7408N, IC144 74151N, IC145 7410N, IC146 7408N, IC147 74257N, IC148 7400N, IC149 74138N, IC15 74257N, IC150 7404N, IC152 74151N, IC153 7432N, IC154 74244N, IC157 74377N, IC158 74377N, IC159 74377N, IC16 74151N, IC160 74151N, IC161 74244N, IC162 74377N, IC163 74244N, IC164 74138N, IC165 74377N, IC166 74377N, IC167 7432N, IC168 7420N, IC169 74377N, IC17 74244N, IC170 74253N, IC171 74377N, IC172 74377N, IC173 7427N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

Commit message: kicad
Connections:
- net data_bus0: no longer IC187.13 (I/O1), IC188.11 (O0), IC208.18 (B1)
- net data_bus1: no longer IC187.14 (I/O2), IC188.12 (O1), IC208.17 (B2)
- net data_bus2: no longer IC187.15 (I/O3), IC188.13 (O2), IC208.16 (B3)
- net data_bus3: no longer IC187.17 (I/O4), IC188.15 (O3), IC208.15 (B4)
- net data_bus4: no longer IC187.18 (I/O5), IC188.16 (O4), IC208.14 (B5)
- net data_bus5: no longer IC187.19 (I/O6), IC188.17 (O5), IC208.13 (B6)
- net data_bus6: no longer IC187.20 (I/O7), IC188.18 (O6), IC208.12 (B7)
- net data_bus7: no longer IC187.21 (I/O8), IC188.19 (O7), IC208.11 (B8)
- net zbus0: now also IC66.3 (1D)
- net zbus1: now also IC66.4 (2D)
- net zbus2: now also IC66.7 (3D)
- net zbus3: now also IC66.8 (4D)
- net zbus4: now also IC66.13 (5D)
- net zbus5: now also IC66.14 (6D)
- net zbus6: now also IC66.17 (7D)
- net zbus7: now also IC66.18 (8D)
- net at IC194.3 (S2), R20.1, S8.1 (O): now also IC194.2 (S1)
- new net: IC187.13 (I/O1), IC188.11 (O0), IC208.18 (B1)
- new net: IC187.14 (I/O2), IC188.12 (O1), IC208.17 (B2)
- new net: IC187.15 (I/O3), IC188.13 (O2), IC208.16 (B3)
- new net: IC187.17 (I/O4), IC188.15 (O3), IC208.15 (B4)
- new net: IC187.18 (I/O5), IC188.16 (O4), IC208.14 (B5)
- new net: IC187.19 (I/O6), IC188.17 (O5), IC208.13 (B6)
- new net: IC187.20 (I/O7), IC188.18 (O6), IC208.12 (B7)
- new net: IC187.21 (I/O8), IC188.19 (O7), IC208.11 (B8)
- no-connect marks 132 -> 133
Other:
- moved on the sheet: IC107A

Commit message: kicad
Parts:
- IC1: footprint main:DIL16 -> Package_DIP:DIP-10_W7.62mm_LongPads
Changed lines of the file:
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@@
       (effects (font (size 1.778 1.5113)) (justify left bottom) hide)
     )
-    (property "Footprint" "main:DIL16" (at 295.91 1921.51 0)
+    (property "Footprint" "Package_DIP:DIP-10_W7.62mm_LongPads" (at 295.91 1921.51 0)
       (effects (font (size 1.27 1.27)) hide)
     )

Commit message: kicad
Parts:
- removed IC150, IC197: 7404N, main:DIL14, symbol main-eagle-import:7404N
- removed IC163: 74244N, main:DIL20, symbol main-eagle-import:74244N
- removed IC195, IC90: 74257N, main:DIL16, symbol main-eagle-import:74257N
- removed IC198: 74377N, main:DIL20, symbol main-eagle-import:74377N
- removed IC218, IC219, IC222, IC223, IC224, IC225, IC228, IC229, IC230, IC27: 74244N, main:DIL20, symbol main-eagle-import:74xx-eu_74244N
- removed S5, S7, S8: tl36po, main:TL3XPO, symbol main-eagle-import:TL36PO
- added IC150, IC163, IC189, IC191, IC195, IC197, IC198, IC200, IC212, IC213: 74244N, main:DIL20, symbol main-eagle-import:74xx-eu_74244N
- added IC151: 74244N, main:DIL20, symbol main-eagle-import:74244N
- added IC155, IC156: 74257N, main:DIL16, symbol main-eagle-import:74257N
- added IC27: 7404N, main:DIL14, symbol main-eagle-import:7404N
- added unit 2 of IC70
- added IC90: 74377N, main:DIL20, symbol main-eagle-import:74377N
- added S1, S2, S3: tl36po, main:TL3XPO, symbol main-eagle-import:TL36PO
Connections:
- net GND: now also IC150.1 (G), IC150.8 (A4), IC151.1 (G), IC151.19 (G), IC163.1 (G), IC189.1 (G), IC191.1 (G), IC195.1 (G), IC197.1 (G), IC198.1 (G), IC198.6 (A3), IC198.8 (A4), IC200.1 (G), IC200.2 (A1), IC200.4 (A2), IC200.6 (A3), IC200.8 (A4), IC212.1 (G), IC213.1 (G), S1.2 (P), S2.2 (P), S3.2 (P)
- net address_bus0: now also IC163.18 (Y1)
- net address_bus1: now also IC163.16 (Y2)
- net address_bus10: now also IC191.14 (Y3)
- net address_bus11: now also IC191.12 (Y4)
- net address_bus12: now also IC195.18 (Y1)
- net address_bus13: now also IC195.16 (Y2)
- net address_bus14: now also IC195.14 (Y3)
- net address_bus15: now also IC195.12 (Y4)
- net address_bus16: now also IC197.18 (Y1)
- net address_bus17: now also IC197.16 (Y2)
- net address_bus18: now also IC197.14 (Y3)
- net address_bus19: now also IC197.12 (Y4)
- net address_bus2: now also IC163.14 (Y3)
- net address_bus20: now also IC198.18 (Y1)
- net address_bus21: now also IC198.16 (Y2)
- net address_bus3: now also IC163.12 (Y4)
- net address_bus4: now also IC189.18 (Y1)
- net address_bus5: now also IC189.16 (Y2)
- net address_bus6: now also IC189.14 (Y3)
- net address_bus7: now also IC189.12 (Y4)
- net address_bus8: now also IC191.18 (Y1)
- net address_bus9: now also IC191.16 (Y2)
- net bus_mem_io: now also IC150.14 (Y3)
- net bus_rd: now also IC150.18 (Y1)
- net bus_tristate: now also IC155.1 (~{A}/B), IC156.1 (~{A}/B)
- net bus_wr: now also IC150.16 (Y2)
- net clk: now also IC90.11 (CLK)
- net data_bus0: now also IC212.18 (Y1)
- net data_bus1: now also IC212.16 (Y2)
- net data_bus2: now also IC212.14 (Y3)
- net data_bus3: now also IC212.12 (Y4)
- net data_bus4: now also IC213.18 (Y1)
- net data_bus5: now also IC213.16 (Y2)
- net data_bus6: now also IC213.14 (Y3)
- net data_bus7: now also IC213.12 (Y4)
- net display_reg_load: now also IC70.3 (I)
- net int_4: now also R22.1; no longer R25.1
- net int_5: now also R25.1; no longer R22.1
- net panel_address_0: now also R37.1, SW7.8, IC163.2 (A1); no longer R29.1, SW6.8
- net panel_address_1: now also R38.1, SW7.7, IC163.4 (A2); no longer R30.1, SW6.7
- net panel_address_10: now also R31.1, SW6.6, IC191.6 (A3); no longer R39.1, SW7.6
- net panel_address_11: now also R32.1, SW6.5, IC191.8 (A4); no longer R40.1, SW7.5
- net panel_address_12: now also R33.1, SW6.4, IC195.2 (A1); no longer R41.1, SW7.4
- net panel_address_13: now also R34.1, SW6.3, IC195.4 (A2); no longer R42.1, SW7.3
- net panel_address_14: now also R35.1, SW6.2, IC195.6 (A3); no longer R43.1, SW7.2
- net panel_address_15: now also R36.1, SW6.1, IC195.8 (A4); no longer R44.1, SW7.1
- net panel_address_16: now also R40.1, IC197.2 (A1); no longer R45.1
- net panel_address_17: now also R42.1, IC197.4 (A2); no longer R46.1
- net panel_address_18: now also R44.1, IC197.6 (A3); no longer R47.1
- net panel_address_19: now also R46.1, IC197.8 (A4); no longer R48.1
- net panel_address_2: now also R39.1, SW7.6, IC163.6 (A3); no longer R31.1, SW6.6
- net panel_address_20: now also R48.1, IC198.2 (A1); no longer R49.1
- net panel_address_21: now also IC198.4 (A2)
- net panel_address_3: now also R41.1, SW7.5, IC163.8 (A4); no longer R32.1, SW6.5
- net panel_address_4: now also R43.1, SW7.4, IC189.2 (A1); no longer R33.1, SW6.4
- net panel_address_5: now also R45.1, SW7.3, IC189.4 (A2); no longer R34.1, SW6.3
- net panel_address_6: now also R47.1, SW7.2, IC189.6 (A3); no longer R35.1, SW6.2
- net panel_address_7: now also R49.1, SW7.1, IC189.8 (A4); no longer R36.1, SW6.1
- net panel_address_8: now also R29.1, SW6.8, IC191.2 (A1); no longer R37.1, SW7.8
- net panel_address_9: now also R30.1, SW6.7, IC191.4 (A2); no longer R38.1, SW7.7
- net panel_data_0: now also IC212.2 (A1)
- net panel_data_1: now also IC212.4 (A2)
- net panel_data_2: now also IC212.6 (A3)
- net panel_data_3: now also IC212.8 (A4)
- net panel_data_4: now also IC213.2 (A1)
- net panel_data_5: now also IC213.4 (A2)
- net panel_data_6: now also IC213.6 (A3)
- net panel_data_7: now also IC213.8 (A4)
- net panel_mem_io: now also IC192.4 (Q), IC150.6 (A3); no longer IC194.4 (Q)
- net panel_rd: now also IC193.4 (Q), IC150.2 (A1); no longer IC192.4 (Q)
- net panel_regsel_0: now also R13.1; no longer R6.1
- net panel_regsel_1: now also R12.1; no longer R7.1
- net panel_regsel_2: now also R11.1; no longer R8.1
- net panel_regsel_3: now also R10.1; no longer R9.1
- net panel_regsel_4: now also R9.1; no longer R10.1
- net panel_wr: now also IC194.4 (Q), IC150.4 (A2); no longer IC193.4 (Q)
- net rd: now also IC27.9 (I); no longer IC70.9 (I)
- net w0: now also IC151.2 (A1), IC90.3 (1D)
- net w1: now also IC151.4 (A2), IC90.4 (2D)
- net w2: now also IC151.6 (A3), IC90.7 (3D)
- net w3: now also IC151.8 (A4), IC90.8 (4D)
- net w4: now also IC151.11 (A1), IC90.13 (5D)
- net w5: now also IC151.13 (A2), IC90.14 (6D)
- net w6: now also IC151.15 (A3), IC90.17 (7D)
- net w7: now also IC151.17 (A4), IC90.18 (8D)
- net wr: now also IC70.9 (I)
- net at IC194.2 (S1), IC194.3 (S2): now also R21.1, S3.1 (O); no longer R20.1
- net at IC192.2 (S1), IC192.3 (S2): now also R19.1, S1.1 (O); no longer R16.1
- net at R17.1: now also IC193.1 (R), S2.3 (S); no longer IC192.1 (R)
- net at IC193.2 (S1), IC193.3 (S2): now also R20.1, S2.1 (O); no longer R18.1
- net at IC194.1 (R): now also R18.1, S3.3 (S); no longer R21.1
- net at IC154.2 (A1): now also IC27.8 (O); no longer IC70.8 (O)
- net at SW4.8: now also R6.1; no longer R13.1
- net at SW4.6: now also R8.1; no longer R11.1
- net at SW4.7: now also R7.1; no longer R12.1
- net at IC154.4 (A2): now also IC70.8 (O)
- new net: IC70.4 (O), IC90.1 (G)
- new net: IC156.2 (1A), IC90.12 (5Q)
- new net: IC156.5 (2A), IC90.15 (6Q)
- new net: IC156.11 (3A), IC90.16 (7Q)
- new net: IC156.14 (4A), IC90.19 (8Q)
- new net: IC155.2 (1A), IC90.2 (1Q)
- new net: IC155.5 (2A), IC90.5 (2Q)
- new net: IC155.11 (3A), IC90.6 (3Q)
- new net: IC155.14 (4A), IC90.9 (4Q)
- new net: IC151.14 (Y3), IC155.10 (3B)
- new net: IC151.12 (Y4), IC155.13 (4B)
- new net: IC155.15 (G), IC156.15 (G)
- new net: IC151.18 (Y1), IC155.3 (1B)
- new net: IC151.16 (Y2), IC155.6 (2B)
- new net: IC151.3 (Y4), IC156.13 (4B)
- new net: IC151.5 (Y3), IC156.10 (3B)
- new net: IC151.7 (Y2), IC156.6 (2B)
- new net: IC151.9 (Y1), IC156.3 (1B)
- new net: IC192.1 (R), R16.1, S1.3 (S)
Other:
- moved on the sheet: IC115C, IC120A, IC138A, IC174B, IC176D, IC186A, IC190A, IC190B, IC411A, R15, R2, R23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

Commit message: kicad
Parts:
- FLAGS0: footprint main:DIL20 -> Package_DIP:DIP-20_W7.62mm
- IC1: footprint Package_DIP:DIP-10_W7.62mm_LongPads -> Package_DIP:DIP-16_W7.62mm
- IC12, IC130, IC133, IC14, IC141, IC144, IC152, IC16, IC160, IC2, IC20, IC23, IC3, IC42, IC44, IC5, IC53, IC56, IC6, IC61, IC62, IC67, IC68, IC69, IC71, IC80, IC81, IC82, IC84, IC85, IC86, IC87, IC88, IC89, IC9: footprint main:DIL16 -> Package_DIP:DIP-16_W7.62mm

Commit message: kicad
Parts:
- added unit 3 of IC107
- added unit 3 of IC108
- added unit 3 of IC126
- added unit 3 of IC74
- added U10, U9: 16550, Package_DIP:DIP-40_W15.24mm, symbol Interface_UART:16550
Connections:
- net GND: now also IC107.7 (GND), IC108.7 (GND), IC126.7 (GND), IC74.7 (GND), U10.12 (CS0), U10.13 (CS1), U9.12 (CS0), U9.13 (CS1)
- net VCC: now also IC107.14 (VCC), IC108.14 (VCC), IC126.14 (VCC), IC74.14 (VCC)
- net uart_0: now also U9.14 (~{CS2})
- net uart_1: now also U10.14 (~{CS2})
