File: hardware/schematics/kicad/main.kicad_sch (KiCad schematic)
At the start: 341 parts, among them IC1 74257N, IC10 74181N, IC100 74257N, IC101 74377N, IC102 74377N, IC103 74153N, IC104 74257N, IC105 74148N, IC106 74377N, IC107 7474N, IC108 7474N, IC109 74377N, IC11 74181N, IC110 74377N, IC111 74253N, IC112 74257N, IC113 74253N, IC114 74257N, IC115 7404N, IC116 74153N, IC117 74377N, IC118 74257N, IC119 7408N, IC12 74151N, IC120 74244N, IC121 74257N, IC122 74257N, IC123 74377N, IC124 74153N, IC125 74257N, IC126 7474N, IC127 74257N, IC128 74157N, IC129 74157N, IC13 74257N, IC130 74151N, IC131 74157N, IC132 74157N, IC133 74151N, IC134 74273N, IC135 74273N, IC136 74273N, IC137 7474N, IC138 7404N, IC139 7400N, IC14 74151N, IC140 58C256P, IC141 74151N, IC142 74257N, IC143 7408N, IC144 74151N, IC145 7410N, IC146 7408N, IC147 74257N, IC148 7400N, IC149 74138N, IC15 74257N, IC150 74244N, IC151 74244N, IC152 74151N, IC153 7432N, IC154 7404N, IC155 74257N, IC156 74257N, IC157 74377N, IC158 74377N, IC159 74377N, IC16 74151N, IC160 74151N, IC161 74244N, IC162 74377N, IC163 74244N, IC164 74138N, IC165 74377N, IC166 74377N, IC167 7432N, IC168 7420N, IC169 74377N, IC17 74244N, IC170 74253N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

Commit message: kicad
Parts:
- IC10, IC11: footprint main:DIL24-6 -> Package_DIP:DIP-24_W7.62mm
- IC100, IC103, IC105, IC111, IC113, IC116, IC124, IC149, IC164, IC170, IC179, IC180, IC181, IC182, IC192, IC193, IC194, IC206, IC214, IC237, IC241, IC255, IC270, IC29, IC30, IC34, IC35, IC36, IC37, IC38, IC40, IC41, IC411, IC412, IC46, IC47, IC49, IC50, IC51, IC52, IC64, IC73, IC83, IC91, IC92, IC95: footprint main:DIL16 -> Package_DIP:DIP-16_W7.62mm
- IC107, IC108, IC115, IC119, IC126, IC137, IC138, IC139, IC143, IC145, IC146, IC148, IC153, IC154, IC167, IC168, IC173, IC174, IC175, IC176, IC18, IC190, IC196, IC201, IC202, IC203, IC205, IC22, IC236, IC25, IC263, IC43, IC45, IC58, IC59, IC70, IC74, IC93, IC94, IC_02_0, IC_04_2, IC_10_0, IC_86_0, IC_86_1: footprint main:DIL14 -> Package_DIP:DIP-14_W7.62mm
- IC134, IC135, IC136, IC208, IC231, IC259, IC266, IC267, IC32, IC33, IC334, IC336, IC338, IC60, IC75, IC76, IC77, IC78, IC79, IC97: footprint main:DIL20 -> Package_DIP:DIP-20_W7.62mm
- IC187: footprint main:DIL32 -> Package_DIP:DIP-32_W7.62mm
- IC188, IC199, IC227, IC243, IC257, IC258, IC261, IC262, IC264, IC265, IC302, IC303, IC333, IC335, IC337, IC339: footprint main:DIL28 -> Package_DIP:DIP-28_W15.24mm
- INT_STATUS_REG0: footprint main:DIL20 -> Package_DIP:DIP-20_W7.62mm_Socket
- U15: footprint (none) -> Package_DIP:DIP-24_W7.62mm

Commit message: kicad
Parts:
- removed unit 3 of IC107
- removed unit 3 of IC108
- removed unit 3 of IC126
- removed IC187: 431000, Package_DIP:DIP-32_W7.62mm, symbol main-eagle-import:431000
- removed unit 3 of IC74
- removed R1, R10, R11, R12, R13, R14, R15, R16, R17, R18, R19, R2, R20, R21, R22, R23, R24, R25, R26, R27, R28, R29, R3, R30, R31, R32, R33, R34, R35, R36, R37, R38, R39, R4, R40, R41, R42, R43, R44, R45, R46, R47, R48, R49, R5, R50, R51, R52, R53, R54, R55, R56, R57, R58, R59, R6, R60, R7, R8, R9: R-US_0204/2V, main:0204V, symbol main-eagle-import:R-US_0204/2V
- removed S1, S2, S3: tl36po, main:TL3XPO, symbol main-eagle-import:TL36PO
- removed SW1, SW2, SW3, SW4, SW5, SW6, SW7, SW8, SW9: SW_DIP-8, main:EDG-08, symbol main-eagle-import:SW_DIP-8
- added RN1, RN2, RN3, RN4, RN5, RN6, RN7, RN8, RN9: R_Pack08, Package_DIP:DIP-16_W7.62mm, symbol Device:R_Pack08
- added SW1, SW10, SW2, SW3, SW4, SW5, SW6, SW7, SW8, SW9: SW_DIP_x08, Package_DIP:DIP-16_W7.62mm, symbol Switch:SW_DIP_x08
- added U15: KM62256CLP, Package_DIP:DIP-28_W15.24mm, symbol Memory_RAM:KM62256CLP
- BIOS_ROM1: renamed from IC188; footprint Package_DIP:DIP-28_W15.24mm -> Package_DIP:DIP-32_W15.24mm
- IC111: renamed from IC125; footprint Package_DIP:DIP-18_W7.62mm -> Package_DIP:DIP-16_W7.62mm
- IC112: renamed from IC118; footprint Package_DIP:DIP-18_W7.62mm -> Package_DIP:DIP-16_W7.62mm
- IC12: renamed from IC13; footprint Package_DIP:DIP-18_W7.62mm -> Package_DIP:DIP-16_W7.62mm
- IC15: renamed from IC98; footprint Package_DIP:DIP-18_W7.62mm -> Package_DIP:DIP-16_W7.62mm
- IC155, IC156: footprint Package_DIP:DIP-18_W7.62mm -> Package_DIP:DIP-16_W7.62mm
- IC157: renamed from IC114; footprint Package_DIP:DIP-18_W7.62mm -> Package_DIP:DIP-16_W7.62mm
- IC158: renamed from IC112; footprint Package_DIP:DIP-18_W7.62mm -> Package_DIP:DIP-16_W7.62mm
- IC159: renamed from IC39; footprint Package_DIP:DIP-18_W7.62mm -> Package_DIP:DIP-16_W7.62mm
- IC16: renamed from IC122; footprint Package_DIP:DIP-18_W7.62mm -> Package_DIP:DIP-16_W7.62mm
- IC160: renamed from IC104; footprint Package_DIP:DIP-18_W7.62mm -> Package_DIP:DIP-16_W7.62mm
- IC177: renamed from IC140; footprint main:DIL28-6 -> Package_DIP:DIP-28_W7.62mm
- IC178: renamed from IC21; footprint main:DIL28-6 -> Package_DIP:DIP-28_W7.62mm
- IC181: renamed from IC131; footprint Package_DIP:DIP-18_W7.62mm -> Package_DIP:DIP-16_W7.62mm
- IC182: renamed from IC128; footprint Package_DIP:DIP-18_W7.62mm -> Package_DIP:DIP-16_W7.62mm
- IC183: renamed from IC129; footprint Package_DIP:DIP-18_W7.62mm -> Package_DIP:DIP-16_W7.62mm
- IC184: renamed from IC132; footprint Package_DIP:DIP-18_W7.62mm -> Package_DIP:DIP-16_W7.62mm
- IC19: renamed from IC121; footprint Package_DIP:DIP-18_W7.62mm -> Package_DIP:DIP-16_W7.62mm
- IC190: renamed from IC142; footprint Package_DIP:DIP-18_W7.62mm -> Package_DIP:DIP-16_W7.62mm
- IC191: renamed from IC147; footprint Package_DIP:DIP-18_W7.62mm -> Package_DIP:DIP-16_W7.62mm
- IC20: renamed from IC127; footprint Package_DIP:DIP-18_W7.62mm -> Package_DIP:DIP-16_W7.62mm
- IC25: renamed from IC55; footprint Package_DIP:DIP-18_W7.62mm -> Package_DIP:DIP-16_W7.62mm
- IC26: renamed from IC63; footprint Package_DIP:DIP-18_W7.62mm -> Package_DIP:DIP-16_W7.62mm
- IC30: renamed from IC15; footprint Package_DIP:DIP-18_W7.62mm -> Package_DIP:DIP-16_W7.62mm
- IC76: renamed from IC341; footprint Package_DIP:DIP-18_W7.62mm -> Package_DIP:DIP-16_W7.62mm
- IRQ_STATUS_1: renamed from INT_STATUS_REG0; footprint Package_DIP:DIP-20_W7.62mm_Socket -> Package_DIP:DIP-20_W7.62mm
- MDR_IN_MUX_1: renamed from IC7; footprint Package_DIP:DIP-18_W7.62mm -> Package_DIP:DIP-16_W7.62mm
- MDR_IN_MUX_2: renamed from IC24; footprint Package_DIP:DIP-18_W7.62mm -> Package_DIP:DIP-16_W7.62mm
- MDR_OUT_MUX_1: renamed from IC54; footprint Package_DIP:DIP-18_W7.62mm -> Package_DIP:DIP-16_W7.62mm
- MDR_OUT_MUX_2: renamed from IC96; footprint Package_DIP:DIP-18_W7.62mm -> Package_DIP:DIP-16_W7.62mm
- U1, U2, U7, U8: footprint main:DIP254P1524X393-32 -> Package_DIP:DIP-32_W15.24mm
- U16: renamed from U15; footprint Package_DIP:DIP-24_W7.62mm -> Package_DIP:DIP-16_W7.62mm
- U3: renamed from U6; footprint main:DIP254P1524X393-32 -> Package_DIP:DIP-32_W15.24mm
- U4: renamed from U3; footprint main:DIP254P1524X393-32 -> Package_DIP:DIP-32_W15.24mm
- U5: renamed from U4; footprint main:DIP254P1524X393-32 -> Package_DIP:DIP-32_W15.24mm
- U6: renamed from U5; footprint main:DIP254P1524X393-32 -> Package_DIP:DIP-32_W15.24mm
- U9: footprint PCDIP24_STM -> Package_DIP:DIP-24_W15.24mm
- renumbered IC11 to ALU_HIGH1, IC10 to ALU_LOW1, FLAGS0 to FLAGS1, IC184 to IC1, IC124 to IC10, IC60 to IC100, IC75 to IC101, IC76 to IC102, IC77 to IC103, IC78 to IC104, IC79 to IC105, IC134 to IC106, IC135 to IC107, IC136 to IC108, IC202 to IC109, IC1 to IC11, IC208 to IC110, IC70 to IC113, IC205 to IC113, IC90 to IC114, IC151 to IC115, IC214 to IC116, IC4 to IC117, IC26 to IC118, IC65 to IC119, IC72 to IC120, IC115 to IC121, IC168 to IC122, IC3 to IC123, IC2 to IC124, IC9 to IC125, IC42 to IC126, IC6 to IC127, IC20 to IC128, IC5 to IC129, IC236 to IC13, IC80 to IC130, IC41 to IC131, IC44 to IC132, IC30 to IC133, IC130 to IC134, IC56 to IC135, IC62 to IC136, IC53 to IC137, IC133 to IC138, IC68 to IC139, IC47 to IC14, IC69 to IC140, IC67 to IC141, IC141 to IC142, IC81 to IC143, IC82 to IC144, IC71 to IC145, IC144 to IC146, IC85 to IC147, IC86 to IC148, IC84 to IC149, IC152 to IC150, IC88 to IC151, IC89 to IC152, IC87 to IC153, IC160 to IC154, IC201 to IC161, IC203 to IC162, IC138 to IC163, IC190 to IC164, IC173 to IC165, IC180 to IC166, IC29 to IC167, IC64 to IC168, IC83 to IC169, IC237 to IC17, IC126 to IC170, IC412 to IC171, IC207 to IC172, IC209 to IC173, IC211 to IC174, IC411 to IC175, IC164 to IC176, IC97 to IC179, IC270 to IC18, IC185 to IC180, IC120 to IC185, IC150 to IC186, IC192 to IC187, IC193 to IC188, IC194 to IC189, IC174 to IC192, IC196 to IC193, IC154 to IC193, IC176 to IC194, IC66 to IC195, IC161 to IC196, IC27 to IC197, IC163 to IC198, IC189 to IC199, IC204 to IC2, IC191 to IC200, IC195 to IC201, IC197 to IC202, IC198 to IC203, IC200 to IC204, IC212 to IC205, IC213 to IC206, IC139 to IC207, IC148 to IC208, IC43 to IC21, IC231 to IC22, IC145 to IC23, IC49 to IC24, IC100 to IC27, IC16 to IC28, IC18 to IC29, IC170 to IC3, IC91 to IC31, IC95 to IC32, IC111 to IC33, IC113 to IC34, IC22 to IC35, IC99 to IC36, IC59 to IC37, IC50 to IC38, IC51 to IC39, IC179 to IC4, IC52 to IC40, IC46 to IC41, IC28 to IC42, IC93 to IC43, IC153 to IC44, IC167 to IC45, IC119 to IC46, IC17 to IC47, IC94 to IC48, IC61 to IC49, IC181 to IC5, IC12 to IC50, IC25 to IC51, IC45 to IC52, IC263 to IC53, IC171 to IC54, IC159 to IC55, IC166 to IC56, IC162 to IC57, IC165 to IC58, IC169 to IC59, IC182 to IC6, IC210 to IC60, IC172 to IC61, IC102 to IC62, IC101 to IC63, IC260 to IC64, IC245 to IC65, IC117 to IC66, IC123 to IC67, IC106 to IC68, IC31 to IC69, IC92 to IC7, IC110 to IC70, IC109 to IC71, IC157 to IC72, IC158 to IC73, IC8 to IC74, IC58 to IC75, IC34 to IC77, IC35 to IC78, IC36 to IC79, IC103 to IC8, IC37 to IC80, IC38 to IC81, IC40 to IC82, IC73 to IC83, IC178 to IC84, IC177 to IC85, IC175 to IC86, IC241 to IC87, IC14 to IC88, IC255 to IC89, IC116 to IC9, IC23 to IC90, IC32 to IC91, IC33 to IC92, IC206 to IC93, IC266 to IC94, IC267 to IC95, IC259 to IC96, IC338 to IC97, IC336 to IC98, IC334 to IC99, IC_02_0 to IC_02_1, IC_04_2 to IC_04_1, IC_10_0 to IC_10_1, IC_86_0 to IC_86_1, IC_86_1 to IC_86_2, IC74 to IRQ_0_DFF1, IC74 to IRQ_1_DFF1, IC107 to IRQ_2_DFF1, IC107 to IRQ_3_DFF1, IC108 to IRQ_4_DFF1, IC108 to IRQ_5_DFF1, IC137 to IRQ_6_DFF1, IC137 to IRQ_7_DFF1, IC146 to IRQ_AND_1, IC143 to IRQ_AND_1, IC146 to IRQ_AND_2, IC143 to IRQ_AND_2, INT_CODE_REG1 to IRQ_CODE1, IC105 to IRQ_ENCODER1, IC149 to IRQ_RST_DECODER1, IC57 to MARH1, IC48 to MARL1, IC183 to MDRH1, IC19 to MDRL1, U12 to U10, U13 to U11, U14 to U12, U10 to U13, U11 to U14, IC264 to U_ROM1, IC243 to U_ROM10, IC257 to U_ROM11, IC261 to U_ROM12, IC262 to U_ROM13, IC302 to U_ROM14, IC303 to U_ROM15, IC265 to U_ROM2, IC258 to U_ROM3, IC339 to U_ROM4, IC337 to U_ROM5, IC335 to U_ROM6, IC333 to U_ROM7, IC227 to U_ROM8, IC199 to U_ROM9
Connections:
- net GND: now also RN8.1 (R1.1), RN8.2 (R2.1), RN8.3 (R3.1), RN8.4 (R4.1), RN8.5 (R5.1), RN8.6 (R6.1), RN8.7 (R7.1), RN8.8 (R8.1), SW1.1, SW1.2, SW1.3, SW1.4, SW1.5, SW1.6, SW1.7, SW1.8, SW3.1, SW3.2, SW3.3, SW3.4, SW3.5, SW3.6, SW3.7, SW3.8, SW4.10, SW4.11, SW4.12, SW4.13, SW4.14, SW4.15, SW4.16, SW4.9, SW6.10, SW6.11, SW6.12, SW6.13, SW6.14, SW6.15, SW6.16, SW6.9, SW7.10, SW7.11, SW7.12, SW7.13, SW7.14, SW7.15, SW7.16, SW7.9, SW8.10, SW8.11, SW8.12, SW8.13, SW8.14, SW8.15, SW8.16, SW8.9, SW9.10, SW9.11, SW9.12, SW9.13, SW9.14, SW9.15, SW9.16, SW9.9, U15.14 (GND)
- net VCC: now also RN1.10 (R7.2), RN1.11 (R6.2), RN1.12 (R5.2), RN1.13 (R4.2), RN1.14 (R3.2), RN1.15 (R2.2), RN1.16 (R1.2), RN1.9 (R8.2), RN2.10 (R7.2), RN2.11 (R6.2), RN2.12 (R5.2), RN2.13 (R4.2), RN2.14 (R3.2), RN2.15 (R2.2), RN2.16 (R1.2), RN2.9 (R8.2), RN3.10 (R7.2), RN3.11 (R6.2), RN3.12 (R5.2), RN3.13 (R4.2), RN3.14 (R3.2), RN3.15 (R2.2), RN3.16 (R1.2), RN3.9 (R8.2), RN4.10 (R7.2), RN4.11 (R6.2), RN4.12 (R5.2), RN4.13 (R4.2), RN4.14 (R3.2), RN4.15 (R2.2), RN4.16 (R1.2), RN4.9 (R8.2), RN5.10 (R7.2), RN5.11 (R6.2), RN5.12 (R5.2), RN5.13 (R4.2), RN5.14 (R3.2), RN5.15 (R2.2), RN5.16 (R1.2), RN5.9 (R8.2), RN6.10 (R7.2), RN6.11 (R6.2), RN6.12 (R5.2), RN6.13 (R4.2), RN6.14 (R3.2), RN6.15 (R2.2), RN6.16 (R1.2), RN6.9 (R8.2), RN7.11 (R6.2), RN7.12 (R5.2), RN7.13 (R4.2), RN7.14 (R3.2), RN7.15 (R2.2), RN7.16 (R1.2), RN9.1 (R1.1), RN9.2 (R2.1), RN9.3 (R3.1), RN9.4 (R4.1), RN9.5 (R5.1), RN9.6 (R6.1), RN9.7 (R7.1), RN9.8 (R8.1), SW10.10, SW10.11, SW10.12, SW10.13, SW10.14, SW10.15, SW10.16, SW10.9, U15.28 (VCC)
- net buffered_rd: now also U15.22 (~{OE})
- net buffered_wr: now also U15.27 (~{WE})
- net clk_crystal: now also SW5.2
- net int_0: now also RN2.1 (R1.1), SW3.16
- net int_1: now also RN2.2 (R2.1), SW3.15
- net int_2: now also RN2.3 (R3.1), SW3.14
- net int_3: now also RN2.4 (R4.1), SW3.13
- net int_4: now also RN2.5 (R5.1), SW3.12
- net int_5: now also RN2.6 (R6.1), SW3.11
- net int_6: now also RN2.7 (R7.1), SW3.10
- net int_7: now also RN2.8 (R8.1), SW3.9
- net panel_address_0: now also RN4.1 (R1.1), SW7.8
- net panel_address_1: now also RN4.2 (R2.1), SW7.7
- net panel_address_10: now also RN3.3 (R3.1), SW6.6
- net panel_address_11: now also RN3.4 (R4.1), SW6.5
- net panel_address_12: now also RN3.5 (R5.1), SW6.4
- net panel_address_13: now also RN3.6 (R6.1), SW6.3
- net panel_address_14: now also RN3.7 (R7.1), SW6.2
- net panel_address_15: now also RN3.8 (R8.1), SW6.1
- net panel_address_16: now also RN5.1 (R1.1), SW8.8
- net panel_address_17: now also RN5.2 (R2.1), SW8.7
- net panel_address_18: now also RN5.3 (R3.1), SW8.6
- net panel_address_19: now also RN5.4 (R4.1), SW8.5
- net panel_address_2: now also RN4.3 (R3.1), SW7.6
- net panel_address_20: now also RN5.5 (R5.1), SW8.4
- net panel_address_21: now also RN5.6 (R6.1), SW8.3
- net panel_address_3: now also RN4.4 (R4.1), SW7.5
- net panel_address_4: now also RN4.5 (R5.1), SW7.4
- net panel_address_5: now also RN4.6 (R6.1), SW7.3
- net panel_address_6: now also RN4.7 (R7.1), SW7.2
- net panel_address_7: now also RN4.8 (R8.1), SW7.1
- net panel_address_8: now also RN3.1 (R1.1), SW6.8
- net panel_address_9: now also RN3.2 (R2.1), SW6.7
- net panel_data_0: now also RN6.1 (R1.1), SW9.8
- net panel_data_1: now also RN6.2 (R2.1), SW9.7
- net panel_data_2: now also RN6.3 (R3.1), SW9.6
- net panel_data_3: now also RN6.4 (R4.1), SW9.5
- net panel_data_4: now also RN6.5 (R5.1), SW9.4
- net panel_data_5: now also RN6.6 (R6.1), SW9.3
- net panel_data_6: now also RN6.7 (R7.1), SW9.2
- net panel_data_7: now also RN6.8 (R8.1), SW9.1
- net panel_regsel_0: now also RN1.8 (R8.1), SW4.1
- net panel_regsel_1: now also RN1.7 (R7.1), SW4.2
- net panel_regsel_2: now also RN1.6 (R6.1), SW4.3
- net panel_regsel_3: now also RN1.5 (R5.1), SW4.4
- net panel_regsel_4: now also RN1.4 (R4.1), SW4.5
- net reset: now also RN9.13 (R4.2), SW1.13
- net rst: now also RN9.12 (R5.2), SW1.16; no longer U11.35 (RESET), U12.35 (RESET), U14.35 (MR)
- net set: now also RN9.14 (R3.2), SW1.14
- net single_step_clk: now also SW5.1
- net stop_clk_req: now also RN9.10 (R7.2), SW1.15
- net at BIOS_ROM1.8 (A2), IC172.14 (Y3): now also U15.8 (A2)
- net at BIOS_ROM1.9 (A1), IC172.16 (Y2): now also U15.9 (A1)
- net at BIOS_ROM1.10 (A0), IC172.18 (Y1): now also U15.10 (A0)
- net at BIOS_ROM1.11 (O0), IC110.18 (B1): now also U15.11 (Q0)
- net at BIOS_ROM1.12 (O1), IC110.17 (B2): now also U15.12 (Q1)
- net at BIOS_ROM1.13 (O2), IC110.16 (B3): now also U15.13 (Q2)
- net at BIOS_ROM1.15 (O3), IC110.15 (B4): now also U15.15 (Q3)
- net at BIOS_ROM1.16 (O4), IC110.14 (B5): now also U15.16 (Q4)
- net at BIOS_ROM1.17 (O5), IC110.13 (B6): now also U15.17 (Q5)
- net at BIOS_ROM1.18 (O6), IC110.12 (B7): now also U15.18 (Q6)
- net at BIOS_ROM1.19 (O7), IC110.11 (B8): now also U15.19 (Q7)
- net at IC122.6 (O): now also U15.20 (~{CS})
- net at BIOS_ROM1.21 (A10), IC162.5 (I4), IC173.14 (Y3): now also U15.21 (A10)
- net at BIOS_ROM1.23 (A11), IC162.4 (I3), IC173.12 (Y4): now also U15.23 (A11)
- net at BIOS_ROM1.24 (A9), IC162.6 (I5), IC173.16 (Y2): now also U15.24 (A9)
- net at BIOS_ROM1.25 (A8), IC162.11 (I6), IC173.18 (Y1): now also U15.25 (A8)
- net at BIOS_ROM1.26 (A13), IC162.2 (I1), IC173.7 (Y2): now also U15.26 (A13)
- net at BIOS_ROM1.27 (A14), IC162.1 (I0), IC173.5 (Y3): now also U15.1 (A14)
- net at BIOS_ROM1.2 (A12), IC162.3 (I2), IC173.9 (Y1): now also U15.2 (A12)
- net at BIOS_ROM1.3 (A7), IC162.12 (I7), IC172.3 (Y4): now also U15.3 (A7)
- net at BIOS_ROM1.4 (A6), IC116.3 (C), IC172.5 (Y3): now also U15.4 (A6)
- net at BIOS_ROM1.5 (A5), IC116.2 (B), IC172.7 (Y2): now also U15.5 (A5)
- net at BIOS_ROM1.6 (A4), IC116.1 (A), IC172.9 (Y1): now also U15.6 (A4)
- net at BIOS_ROM1.7 (A3), IC172.12 (Y4): now also U15.7 (A3)
- net at IC188.1 (R): now also RN7.3 (R3.1), RN8.14 (R3.2), SW10.6
- net at IC121.1 (I), IC171.7 (CLK): now also SW2.10, SW2.11, SW2.12, SW2.13, SW2.14, SW2.15, SW2.16, SW2.9
- net at IC188.2 (S1), IC188.3 (S2): now also RN7.4 (R4.1), RN8.13 (R4.2), SW10.5
- net at IC187.1 (R): now also RN7.5 (R5.1), RN8.11 (R6.2), SW10.3
- net at IC185.2 (A1): now also SW5.10, SW5.11, SW5.12, SW5.13, SW5.14, SW5.15, SW5.16, SW5.9
- net at IC164.12 (D): now also RN9.9 (R8.2), SW1.11
- net at IC164.2 (D): now also RN9.11 (R6.2), SW1.12
- net at IC189.2 (S1), IC189.3 (S2): now also RN7.2 (R2.1), RN8.15 (R2.2), SW10.7
- net at IC189.1 (R): now also RN7.1 (R1.1), RN8.16 (R1.2), SW10.8
- net at IC187.2 (S1), IC187.3 (S2): now also RN7.6 (R6.1), RN8.12 (R5.2), SW10.4
- net at U16.9 (Q0): now also SW2.1
- net at U16.7 (Q1): now also SW2.2
- net at U16.6 (Q2): now also SW2.3
- net at U16.5 (Q3): now also SW2.4
- net at U16.3 (Q4): now also SW2.5
- net at U16.2 (Q5): now also SW2.6
- net at U16.4 (Q6): now also SW2.7
- net at U16.13 (Q7): now also SW2.8
- new net: RN1.3 (R3.1), SW4.6
- new net: RN1.2 (R2.1), SW4.7
- new net: RN1.1 (R1.1), SW4.8
- new net: RN5.8 (R8.1), SW8.1
- new net: RN5.7 (R7.1), SW8.2
- no-connect marks 159 -> 165
Other:
- note added: "IMPROVE THIS PART OF THE CIRCUIT"
- moved on the sheet: IC187A, IC188A, IC189A, U16, X1

Commit message: kicad
Parts:
- renumbered IC46 to IC13, IC43 to IC13, IC52 to IC13, IC86 to IC37
Connections:
- net any_interruption: now also IC13.10 (I1); no longer IC13.2 (I1)
- net cond_invert: now also IC37.1 (I0); no longer IC37.4 (I0)
- net condition: now also IC37.2 (I1); no longer IC37.5 (I1)
- net final_condition: now also IC37.3 (O); no longer IC37.6 (O)
- net mux_a: now also IC13.11 (O); no longer IC13.3 (O)
- net mux_b: now also IC13.6 (O); no longer IC13.3 (O)
- net typ_1: now also IC13.12 (I0), IC13.4 (I0); no longer IC13.1 (I0), IC13.1 (I0)
- net at IC48.5 (I1): now also IC13.8 (O); no longer IC13.3 (O)
- net at IC48.6 (O): now also IC13.13 (I1); no longer IC13.2 (I1)
- new net: IC13.5 (I1), IC13.9 (I0), IC21.8 (O)
Other:
- moved on the sheet: IC29A, IC29B, IC29C, IC35A

Commit message: kicad
Parts:
- added unit 2 of IC91
- added unit 2 of IC92
Connections:
- net GND: now also IC91.10 (GND), IC92.10 (GND)
- net VCC: now also IC91.20 (VCC), IC92.20 (VCC)
Changed lines of the file:
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@@
     )
   )
+  (symbol (lib_id "main-eagle-import:74273N") (at 783.59 1159.51 0) (unit 2)
+    (in_bom yes) (on_board yes) (dnp no)
+    (property "Reference" "IC91" (at 782.955 1158.875 0)
+      (effects (font (size 1.778 1.5113)) (justify left bottom))
+    )
+    (property "Value" "74273N" (at 775.97 1177.29 0)
+      (effects (font (size 1.778 1.5113)) (justify left bottom) hide)
+    )
+    (property "Footprint" "Package_DIP:DIP-20_W7.62mm" (at 783.59 1159.51 0)
+      (effects (font (size 1.27 1.27)) hide)
+    )
+    (property "Datasheet" "" (at 783.59 1159.51 0)
+      (effects (font (size 1.27 1.27)) hide)
+    )
+    (property "OC_FARNELL" "unknown" (at 783.59 1159.51 0)
+      (effects (font (size 1.27 1.27)) (justify right top) hide)
+    )
+    (pin "1")
+    (pin "11")
+    (pin "12")
+    (pin "13")
+    (pin "14")
+    (pin "15")
+    (pin "16")
+    (pin "17")
+    (pin "18")
+    (pin "19")
+    (pin "2")
+    (pin "3")
+    (pin "4")
+    (pin "5")
+    (pin "6")
+    (pin "7")
+    (pin "8")
+    (pin "9")
+    (pin "10")
+    (pin "20")
+    (instances
+      (project "main"
+        (path "/8dc530de-176d-4542-9ed1-97157904b8fd"
+          (reference "IC91") (unit 2)
+        )
+      )
+    )
+  )
   (symbol (lib_id "main-eagle-import:GND") (at 1390.65 1398.27 0) (unit 1)
     (in_bom yes) (on_board yes) (dnp no)
@@
     )
   )
+  (symbol (lib_id "main-eagle-import:74273N") (at 792.48 1159.51 0) (unit 2)
+    (in_bom yes) (on_board yes) (dnp no)
+    (property "Reference" "IC92" (at 791.845 1160.145 0)
+      (effects (font (size 1.778 1.5113)) (justify left bottom))
+    )
+    (property "Value" "74273N" (at 784.86 1177.29 0)
+      (effects (font (size 1.778 1.5113)) (justify left bottom) hide)
+    )
+    (property "Footprint" "Package_DIP:DIP-20_W7.62mm" (at 792.48 1159.51 0)
+      (effects (font (size 1.27 1.27)) hide)
+    )
+    (property "Datasheet" "" (at 792.48 1159.51 0)
+      (effects (font (size 1.27 1.27)) hide)
+    )
+    (property "OC_FARNELL" "unknown" (at 792.48 1159.51 0)
+      (effects (font (size 1.27 1.27)) (justify right top) hide)
+    )
+    (pin "1")
+    (pin "11")
+    (pin "12")
+    (pin "13")
+    (pin "14")
+    (pin "15")
+    (pin "16")
+    (pin "17")
+    (pin "18")
+    (pin "19")
+    (pin "2")
+    (pin "3")
+    (pin "4")
+    (pin "5")
+    (pin "6")
+    (pin "7")
+    (pin "8")
+    (pin "9")
+    (pin "10")
+    (pin "20")
+    (instances
+      (project "main"
+        (path "/8dc530de-176d-4542-9ed1-97157904b8fd"
+          (reference "IC92") (unit 2)
+        )
+      )
+    )
+  )
   (symbol (lib_id "main-eagle-import:74151N") (at 1184.91 2792.73 0) (unit 1)
     (in_bom yes) (on_board yes) (dnp no)
@@
     )
   )
+  (symbol (lib_id "power:GND") (at 783.59 1169.67 0) (unit 1)
+    (in_bom yes) (on_board yes) (dnp no)
+    (property "Reference" "#PWR0124" (at 783.59 1176.02 0)
+      (effects (font (size 1.27 1.27)) hide)
+    )
+    (property "Value" "GND" (at 783.59 1170.94 0)
+      (effects (font (size 1.27 1.27)))
+    )
+    (property "Footprint" "" (at 783.59 1169.67 0)
+      (effects (font (size 1.27 1.27)) hide)
+    )
+    (property "Datasheet" "" (at 783.59 1169.67 0)
+      (effects (font (size 1.27 1.27)) hide)
+    )
+    (pin "1")
+    (instances
+      (project "main"
+        (path "/8dc530de-176d-4542-9ed1-97157904b8fd"
+          (reference "#PWR0124") (unit 1)
+        )
+      )
+    )
+  )
   (symbol (lib_id "main-eagle-import:GND") (at 1501.14 519.43 0) (unit 1)
     (in_bom yes) (on_board yes) (dnp no)
@@
     )
   )
+  (symbol (lib_id "power:VCC") (at 783.59 1149.35 0) (unit 1)
+    (in_bom yes) (on_board yes) (dnp no) (fields_autoplaced)
+    (property "Reference" "#PWR0125" (at 783.59 1153.16 0)
+      (effects (font (size 1.27 1.27)) hide)
+    )
+    (property "Value" "VCC" (at 783.59 1144.27 0)
+      (effects (font (size 1.27 1.27)))
+    )
+    (property "Footprint" "" (at 783.59 1149.35 0)
+      (effects (font (size 1.27 1.27)) hide)
+    )
+    (property "Datasheet" "" (at 783.59 1149.35 0)
+      (effects (font (size 1.27 1.27)) hide)
+    )
+    (pin "1")
+    (instances
+      (project "main"
+        (path "/8dc530de-176d-4542-9ed1-97157904b8fd"
+          (reference "#PWR0125") (unit 1)
+        )
+      )
+    )
+  )
   (symbol (lib_id "main-eagle-import:74283N") (at 580.39 1339.85 0) (unit 1)
     (in_bom yes) (on_board yes) (dnp no)
@@
     )
   )
+  (symbol (lib_id "power:VCC") (at 792.48 1149.35 0) (unit 1)
+    (in_bom yes) (on_board yes) (dnp no) (fields_autoplaced)
+    (property "Reference" "#PWR0139" (at 792.48 1153.16 0)
+      (effects (font (size 1.27 1.27)) hide)
+    )
+    (property "Value" "VCC" (at 792.48 1144.27 0)
+      (effects (font (size 1.27 1.27)))
+    )
+    (property "Footprint" "" (at 792.48 1149.35 0)
+      (effects (font (size 1.27 1.27)) hide)
+    )
+    (property "Datasheet" "" (at 792.48 1149.35 0)
+      (effects (font (size 1.27 1.27)) hide)
+    )
+    (pin "1")
+    (instances
+      (project "main"
+        (path "/8dc530de-176d-4542-9ed1-97157904b8fd"
+          (reference "#PWR0139") (unit 1)
+        )
+      )
+    )
+  )
   (symbol (lib_id "main-eagle-import:74153N") (at 775.97 2007.87 0) (unit 1)
     (in_bom yes) (on_board yes) (dnp no)
@@
         )
       )
+    )
+  )
+  (symbol (lib_id "power:GND") (at 792.48 1169.67 0) (unit 1)
+    (in_bom yes) (on_board yes) (dnp no)
+    (property "Reference" "#PWR0140" (at 792.48 1176.02 0)
+      (effects (font (size 1.27 1.27)) hide)
+    )
+    (property "Value" "GND" (at 792.48 1170.94 0)
+      (effects (font (size 1.27 1.27)))
+    )
+    (property "Footprint" "" (at 792.48 1169.67 0)
+      (effects (font (size 1.27 1.27)) hide)
+    )
+    (property "Datasheet" "" (at 792.48 1169.67 0)
+      (effects (font (size 1.27 1.27)) hide)
+    )
+    (pin "1")
+    (instances
+      (project "main"
+        (path "/8dc530de-176d-4542-9ed1-97157904b8fd"
+          (reference "#PWR0140") (unit 1)
+        )
+      )

Commit message: kicad
Parts:
- removed unit 3 of IC_10_1
- added IC_10_2: 7410N, Package_DIP:DIP-14_W7.62mm, symbol main-eagle-import:7410N
Connections:
- net buffered_mem_io: now also IC_10_2.11 (I2)
- net at IC122.2 (I1), IC161.3 (O): now also IC_10_2.10 (I1)
- net at IC113.2 (O): now also IC_10_2.9 (I0)
- net at BIOS_ROM1.20 (~{CE}): now also IC_10_2.8 (O)
Changed lines of the file:
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@@
     )
   )
-  (symbol (lib_id "main-eagle-import:7410N") (at 1182.37 694.69 180) (unit 3)
-    (in_bom yes) (on_board yes) (dnp no)
-    (property "Reference" "IC_10_1" (at 1183.005 694.055 0)
-      (effects (font (size 1.778 1.5113)) (justify left bottom))
-    )
-    (property "Value" "7410N" (at 1189.99 687.07 0)
-      (effects (font (size 1.778 1.5113)) (justify left bottom) hide)
-    )
-    (property "Footprint" "Package_DIP:DIP-14_W7.62mm" (at 1182.37 694.69 0)
-      (effects (font (size 1.27 1.27)) hide)
-    )
-    (property "Datasheet" "" (at 1182.37 694.69 0)
-      (effects (font (size 1.27 1.27)) hide)
-    )
-    (pin "1")
-    (pin "12")
-    (pin "13")
-    (pin "2")
-    (pin "3")
-    (pin "4")
-    (pin "5")
-    (pin "6")
-    (pin "10")
-    (pin "11")
-    (pin "8")
-    (pin "9")
-    (pin "14")
-    (pin "7")
-    (instances
-      (project "main"
-        (path "/8dc530de-176d-4542-9ed1-97157904b8fd"
-          (reference "IC_10_1") (unit 3)
-        )
-      )
-    )
-  )
   (symbol (lib_id "main-eagle-import:74157N") (at 1342.39 1690.37 0) (unit 1)
     (in_bom yes) (on_board yes) (dnp no)
@@
         )
       )
+    )
+  )
+  (symbol (lib_id "main-eagle-import:7410N") (at 1182.37 694.69 180) (unit 3)
+    (in_bom yes) (on_board yes) (dnp no)
+    (property "Reference" "IC_10_2" (at 1183.005 694.055 0)
+      (effects (font (size 1.778 1.5113)) (justify left bottom))
+    )
+    (property "Value" "7410N" (at 1189.99 687.07 0)
+      (effects (font (size 1.778 1.5113)) (justify left bottom) hide)
+    )
+    (property "Footprint" "Package_DIP:DIP-14_W7.62mm" (at 1182.37 694.69 0)
+      (effects (font (size 1.27 1.27)) hide)
+    )
+    (property "Datasheet" "" (at 1182.37 694.69 0)
+      (effects (font (size 1.27 1.27)) hide)
+    )
+    (pin "1")
+    (pin "12")
+    (pin "13")
+    (pin "2")
+    (pin "3")
+    (pin "4")
+    (pin "5")
+    (pin "6")
+    (pin "10")
+    (pin "11")
+    (pin "8")
+    (pin "9")
+    (pin "14")
+    (pin "7")
+    (instances
+      (project "main"
+        (path "/8dc530de-176d-4542-9ed1-97157904b8fd"
+          (reference "IC_10_2") (unit 3)
+        )
+      )
