File: hardware/schematics/kicad/_autosave-main.kicad_sch (KiCad schematic)
At the start: 341 parts, among them IC1 74257N, IC10 74181N, IC100 74257N, IC101 74377N, IC102 74377N, IC103 74153N, IC104 74257N, IC105 74148N, IC106 74377N, IC107 7474N, IC108 7474N, IC109 74377N, IC11 74181N, IC110 74377N, IC111 74253N, IC112 74257N, IC113 74253N, IC114 74257N, IC115 7404N, IC116 74153N, IC117 74377N, IC118 74257N, IC119 7408N, IC12 74151N, IC120 74244N, IC121 74257N, IC122 74257N, IC123 74377N, IC124 74153N, IC125 74257N, IC126 7474N, IC127 74257N, IC128 74157N, IC129 74157N, IC13 74257N, IC130 74151N, IC131 74157N, IC132 74157N, IC133 74151N, IC134 74273N, IC135 74273N, IC136 74273N, IC137 7474N, IC138 7404N, IC139 7400N, IC14 74151N, IC140 58C256P, IC141 74151N, IC142 74257N, IC143 7408N, IC144 74151N, IC145 7410N, IC146 7408N, IC147 74257N, IC148 7400N, IC149 74138N, IC15 74257N, IC150 74244N, IC151 74244N, IC152 74151N, IC153 7432N, IC154 7404N, IC155 74257N, IC156 74257N, IC157 74377N, IC158 74377N, IC159 74377N, IC16 74151N, IC160 74151N, IC161 74244N, IC162 74377N, IC163 74244N, IC164 74138N, IC165 74377N, IC166 74377N, IC167 7432N, IC168 7420N, IC169 74377N, IC17 74244N, IC170 74253N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

Commit message: kicad
Parts:
- IC10, IC11: footprint main:DIL24-6 -> Package_DIP:DIP-24_W7.62mm
- IC100, IC103, IC105, IC111, IC113, IC116, IC124, IC149, IC164, IC170, IC179, IC180, IC181, IC182, IC192, IC193, IC194, IC206, IC214, IC237, IC241, IC255, IC270, IC29, IC30, IC34, IC35, IC36, IC37, IC38, IC40, IC41, IC411, IC412, IC46, IC47, IC49, IC50, IC51, IC52, IC64, IC73, IC83, IC91, IC92, IC95: footprint main:DIL16 -> Package_DIP:DIP-16_W7.62mm
- IC107, IC108, IC115, IC119, IC126, IC137, IC138, IC139, IC143, IC145, IC146, IC148, IC153, IC154, IC167, IC168, IC173, IC174, IC175, IC176, IC18, IC190, IC196, IC201, IC202, IC203, IC205, IC22, IC236, IC25, IC263, IC43, IC45, IC58, IC59, IC70, IC74, IC93, IC94, IC_02_0, IC_04_2, IC_10_0, IC_86_0, IC_86_1: footprint main:DIL14 -> Package_DIP:DIP-14_W7.62mm
- U15: footprint (none) -> Package_DIP:DIP-24_W7.62mm
