File: hardware/schematics/kicad/_autosave-main.kicad_sch (KiCad schematic)
At the start: 288 parts, among them IC1 74377N, IC10 74153N, IC100 74273N, IC101 74273N, IC102 74273N, IC103 74273N, IC104 74273N, IC105 74273N, IC106 74273N, IC107 74273N, IC108 74273N, IC109 7427N, IC11 74257N, IC110 74245N, IC111 74257N, IC112 74257N, IC113 7404N, IC114 74377N, IC115 74244N, IC116 74138N, IC117 74244N, IC118 74244N, IC119 74244N, IC12 74257N, IC120 74244N, IC121 7404N, IC122 7420N, IC123 74151N, IC124 74151N, IC125 74151N, IC126 74151N, IC127 74151N, IC128 74151N, IC129 74151N, IC13 7408N, IC130 74151N, IC131 74151N, IC132 74151N, IC133 74151N, IC134 74151N, IC135 74151N, IC136 74151N, IC137 74151N, IC138 74151N, IC139 74151N, IC14 74153N, IC140 74151N, IC141 74151N, IC142 74151N, IC143 74151N, IC144 74151N, IC145 74151N, IC146 74151N, IC147 74151N, IC148 74151N, IC149 74151N, IC15 74257N, IC150 74151N, IC151 74151N, IC152 74151N, IC153 74151N, IC154 74151N, IC155 74257N, IC156 74257N, IC157 74257N, IC158 74257N, IC159 74257N, IC16 74257N, IC160 74257N, IC161 7408N, IC162 7430N, IC163 7404N, IC164 7474N, IC165 7427N, IC166 74153N, IC167 74153N, IC168 74153N, IC169 74153N, IC17 74153N, IC170 7474N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

Commit message: kicad
Parts:
- ALU_HIGH1, ALU_LOW1: footprint Package_DIP:DIP-24_W7.62mm -> main:DIL24-6
- BIOS_ROM1: footprint Package_DIP:DIP-32_W15.24mm -> main:DIL28
- FLAGS1, IC1, IC100, IC101, IC102, IC103, IC104, IC105, IC106, IC107, IC108, IC110, IC114, IC115, IC117, IC118, IC119, IC120, IC172, IC173, IC174, IC179, IC180, IC185, IC186, IC195, IC196, IC197, IC198, IC199, IC2, IC200, IC201, IC202, IC203, IC204, IC205, IC206, IC22, IC36, IC42, IC47, IC54, IC55, IC56, IC57, IC58, IC59, IC60, IC61, IC62, IC63, IC64, IC65, IC66, IC67, IC68, IC69, IC70, IC71, IC72, IC73, IC74, IC84, IC85, IC91, IC92, IC94, IC95, IC96, IC97, IC98, IC99, IRQ_CODE1, IRQ_STATUS_1, MARH1, MARL1, MDRH1, MDRL1: footprint Package_DIP:DIP-20_W7.62mm -> main:DIL20
- IC10, IC11, IC111, IC112, IC116, IC12, IC123, IC124, IC125, IC126, IC127, IC128, IC129, IC130, IC131, IC132, IC133, IC134, IC135, IC136, IC137, IC138, IC139, IC14, IC140, IC141, IC142, IC143, IC144, IC145, IC146, IC147, IC148, IC149, IC15, IC150, IC151, IC152, IC153, IC154, IC155, IC156, IC157, IC158, IC159, IC16, IC160, IC166, IC167, IC168, IC169, IC17, IC175, IC176, IC18, IC181, IC182, IC183, IC184, IC187, IC188, IC189, IC19, IC190, IC191, IC20, IC24, IC25, IC26, IC27, IC28, IC3, IC30, IC31, IC32, IC33, IC34, IC38, IC39, IC4, IC40, IC41, IC49, IC5, IC50, IC6, IC7, IC76, IC77, IC78, IC79, IC8, IC80, IC81, IC82, IC83, IC87, IC88, IC89, IC9, IC90, IC93, IRQ_ENCODER1, IRQ_RST_DECODER1, MDR_IN_MUX_1, MDR_IN_MUX_2, MDR_OUT_MUX_1, MDR_OUT_MUX_2: footprint Package_DIP:DIP-16_W7.62mm -> main:DIL16
- IC109, IC113, IC121, IC122, IC13, IC161, IC162, IC163, IC164, IC165, IC170, IC192, IC193, IC194, IC207, IC208, IC21, IC23, IC29, IC35, IC37, IC44, IC45, IC48, IC51, IC53, IC75, IC_02_1, IC_04_1, IC_10_1, IC_10_2, IC_86_1, IC_86_2, IRQ_0_DFF1, IRQ_1_DFF1, IRQ_2_DFF1, IRQ_3_DFF1, IRQ_4_DFF1, IRQ_5_DFF1, IRQ_6_DFF1, IRQ_7_DFF1, IRQ_AND_1, IRQ_AND_2: footprint Package_DIP:DIP-14_W7.62mm -> main:DIL14
- IC177, IC178: footprint Package_DIP:DIP-28_W7.62mm -> main:DIL28-6
- U1, U2, U3, U4, U5, U6, U7, U8: footprint Package_DIP:DIP-32_W15.24mm -> main:DIP254P1524X393-32
- U_ROM1, U_ROM10, U_ROM11, U_ROM12, U_ROM13, U_ROM14, U_ROM15, U_ROM2, U_ROM3, U_ROM4, U_ROM5, U_ROM6, U_ROM7, U_ROM8, U_ROM9: footprint Package_DIP:DIP-28_W15.24mm -> main:DIL28
Connections:
- net GND: no longer U18.8 (GND)
- net VCC: no longer U18.16 (VCC)
