File: hardware/schematics/kicad/_autosave-main.kicad_sch (KiCad schematic)
At the start: 295 parts, among them IC1 74377N, IC10 74153N, IC100 74273N, IC101 74273N, IC102 74273N, IC103 74273N, IC104 74273N, IC105 74273N, IC106 74273N, IC107 74273N, IC108 74273N, IC109 7427N, IC11 74257N, IC110 74245N, IC111 74257N, IC112 74257N, IC113 7404N, IC114 74377N, IC115 74244N, IC116 74138N, IC117 74244N, IC118 74244N, IC119 74244N, IC12 74257N, IC120 74244N, IC121 7404N, IC122 7420N, IC123 74151N, IC124 74151N, IC125 74151N, IC126 74151N, IC127 74151N, IC128 74151N, IC129 74151N, IC13 7408N, IC130 74151N, IC131 74151N, IC132 74151N, IC133 74151N, IC134 74151N, IC135 74151N, IC136 74151N, IC137 74151N, IC138 74151N, IC139 74151N, IC14 74153N, IC140 74151N, IC141 74151N, IC142 74151N, IC143 74151N, IC144 74151N, IC145 74151N, IC146 74151N, IC147 74151N, IC148 74151N, IC149 74151N, IC15 74257N, IC150 74151N, IC151 74151N, IC152 74151N, IC153 74151N, IC154 74151N, IC155 74257N, IC156 74257N, IC157 74257N, IC158 74257N, IC159 74257N, IC16 74257N, IC160 74257N, IC161 7408N, IC162 7430N, IC163 7404N, IC164 7474N, IC165 7427N, IC166 74153N, IC167 74153N, IC168 74153N, IC169 74153N, IC17 74153N, IC170 7474N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

Commit message: floppy
Connections:
- net index: now also RN9.15 (R2.2); no longer RN9.16 (R1.2)
- net track_0: now also RN9.14 (R3.2); no longer RN9.15 (R2.2)
- net write_protect: now also RN9.16 (R1.2); no longer RN9.14 (R3.2)
Changed lines of the file:
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@@
 	)
 	(junction
+		(at 1584.96 642.62)
+		(diameter 0)
+		(color 0 0 0 0)
+	)
+	(junction
 		(at 852.17 2284.73)
 		(diameter 0)
@@
 	)
 	(junction
+		(at 1587.5 640.08)
+		(diameter 0)
+		(color 0 0 0 0)
+	)
+	(junction
 		(at 728.98 1418.59)
 		(diameter 0)
@@
 	)
 	(junction
-		(at 1584.96 637.54)
-		(diameter 0)
-		(color 0 0 0 0)
-	)
-	(junction
 		(at 627.38 1631.95)
 		(diameter 0)
@@
 	)
 	(junction
-		(at 1587.5 642.62)
-		(diameter 0)
-		(color 0 0 0 0)
-	)
-	(junction
 		(at 1158.24 1352.55)
 		(diameter 0)
@@
 	)
 	(junction
-		(at 1590.04 640.08)
-		(diameter 0)
-		(color 0 0 0 0)
-	)
-	(junction
 		(at 1744.98 1892.3)
 		(diameter 0)
@@
 	)
 	(junction
+		(at 1590.04 637.54)
+		(diameter 0)
+		(color 0 0 0 0)
+	)
+	(junction
 		(at 1605.28 2555.24)
 		(diameter 0)
@@
 	(wire
 		(pts
+			(xy 1587.5 610.87) (xy 1587.5 640.08)
+		)
+		(stroke
+			(width 0)
+			(type default)
+		)
+	)
+	(wire
+		(pts
 			(xy 1826.26 2446.02) (xy 1778 2446.02)
 		)
@@
 		)
 	)
+	(wire
+		(pts
+			(xy 1590.04 637.54) (xy 1592.58 637.54)
+		)
+		(stroke
+			(width 0)
+			(type default)
+		)
+	)
 	(bus
 		(pts
@@
 	(wire
 		(pts
+			(xy 1579.88 610.87) (xy 1579.88 621.03)
+		)
+		(stroke
+			(width 0)
+			(type default)
+		)
+	)
+	(wire
+		(pts
 			(xy 1934.21 1007.11) (xy 1936.75 1007.11)
 		)
@@
 		)
 	)
-	(wire
-		(pts
-			(xy 1550.67 642.62) (xy 1587.5 642.62)
-		)
-		(stroke
-			(width 0)
-			(type default)
-		)
-	)
 	(bus
 		(pts
@@
 	(wire
 		(pts
+			(xy 1590.04 610.87) (xy 1590.04 637.54)
+		)
+		(stroke
+			(width 0)
+			(type default)
+		)
+	)
+	(wire
+		(pts
 			(xy 852.17 2371.09) (xy 868.68 2371.09)
 		)
@@
 		)
 	)
-	(wire
-		(pts
-			(xy 1579.88 610.87) (xy 1579.88 621.03)
-		)
-		(stroke
-			(width 0)
-			(type default)
-		)
-	)
 	(bus
 		(pts
@@
 	(wire
 		(pts
+			(xy 1584.96 642.62) (xy 1592.58 642.62)
+		)
+		(stroke
+			(width 0)
+			(type default)
+		)
+	)
+	(wire
+		(pts
 			(xy 1877.06 1033.78) (xy 1887.22 1033.78)
 		)
@@
 	(wire
 		(pts
+			(xy 1709.42 497.84) (xy 1711.96 497.84)
+		)
+		(stroke
+			(width 0)
+			(type default)
+		)
+	)
+	(wire
+		(pts
 			(xy 654.05 1149.35) (xy 685.8 1149.35)
 		)
@@
 		)
 	)
-	(wire
-		(pts
-			(xy 1711.96 497.84) (xy 1709.42 497.84)
-		)
-		(stroke
-			(width 0)
-			(type default)
-		)
-	)
 	(bus
 		(pts
@@
 	(wire
 		(pts
+			(xy 1587.5 640.08) (xy 1592.58 640.08)
+		)
+		(stroke
+			(width 0)
+			(type default)
+		)
+	)
+	(wire
+		(pts
 			(xy 1715.77 1534.16) (xy 1715.77 1404.62)
 		)
@@
 	(wire
 		(pts
-			(xy 1584.96 610.87) (xy 1584.96 637.54)
-		)
-		(stroke
-			(width 0)
-			(type default)
-		)
-	)
-	(wire
-		(pts
 			(xy 1021.08 1859.28) (xy 1168.4 1859.28)
 		)
@@
 	(wire
 		(pts
-			(xy 1590.04 610.87) (xy 1590.04 640.08)
-		)
-		(stroke
-			(width 0)
-			(type default)
-		)
-	)
-	(wire
-		(pts
 			(xy 1929.13 1031.24) (xy 1934.21 1031.24)
 		)
@@
 	(wire
 		(pts
-			(xy 1550.67 640.08) (xy 1590.04 640.08)
+			(xy 1550.67 640.08) (xy 1587.5 640.08)
 		)
 		(stroke
@@
 	(wire
 		(pts
-			(xy 1590.04 640.08) (xy 1592.58 640.08)
-		)
-		(stroke
-			(width 0)
-			(type default)
-		)
-	)
-	(wire
-		(pts
 			(xy 1643.38 2501.9) (xy 1630.68 2501.9)
 		)
@@
 	(wire
 		(pts
-			(xy 1587.5 610.87) (xy 1587.5 642.62)
-		)
-		(stroke
-			(width 0)
-			(type default)
-		)
-	)
-	(wire
-		(pts
 			(xy 730.25 2381.25) (xy 707.39 2381.25)
 		)
@@
 	(wire
 		(pts
-			(xy 1550.67 637.54) (xy 1584.96 637.54)
+			(xy 1550.67 637.54) (xy 1590.04 637.54)
 		)
 		(stroke
@@
 		)
 	)
+	(wire
+		(pts
+			(xy 1584.96 610.87) (xy 1584.96 642.62)
+		)
+		(stroke
+			(width 0)
+			(type default)
+		)
+	)
 	(bus
 		(pts
@@
 	(wire
 		(pts
-			(xy 1584.96 637.54) (xy 1592.58 637.54)
-		)
-		(stroke
-			(width 0)
-			(type default)
-		)
-	)
-	(wire
-		(pts
 			(xy 1784.35 1412.24) (xy 1840.23 1412.24)
 		)
@@
 	(wire
 		(pts
-			(xy 1587.5 642.62) (xy 1592.58 642.62)
+			(xy 1550.67 642.62) (xy 1584.96 642.62)
 		)
 		(stroke
