File: hardware/schematics/kicad/main.kicad_pcb (KiCad board)
At the start: 2 copper layers, 37 parts, among them IC1 74257N, IC12 74151N, IC130 74151N, IC133 74151N, IC14 74151N, IC141 74151N, IC144 74151N, IC152 74151N, IC16 74151N, IC160 74151N, IC2 74151N, IC20 74151N, IC23 74151N, IC3 74151N, IC42 74151N, IC44 74151N, IC5 74151N, IC53 74151N, IC56 74151N, IC6 74151N, IC61 74151N, IC62 74151N, IC67 74151N, IC68 74151N, IC69 74151N, IC71 74151N, IC80 74151N, IC81 74151N, IC82 74151N, IC84 74151N, IC85 74151N, IC86 74151N, IC87 74151N, IC88 74151N, IC89 74151N, IC9 74151N

Commit message: kicad
Parts:
- added ALU_HIGH1: 74181N, Package_DIP:DIP-24_W7.62mm, F.Cu at (-333.9, -127.3)
- added ALU_LOW1: 74181N, Package_DIP:DIP-24_W7.62mm, F.Cu at (-344.8, -127.3)
- added BIOS_RAM1: 431000, Package_DIP:DIP-32_W15.24mm, F.Cu at (475.2, 83.5)
- added BIOS_ROM1: 27512, Package_DIP:DIP-32_W15.24mm, F.Cu at (495.8, 83.4)
- added IC100: 74257N, Package_DIP:DIP-16_W7.62mm, F.Cu at (345.0, 149.1)
- added IC101: 74377N, Package_DIP:DIP-20_W7.62mm, F.Cu at (301.6, 263.7)
- added IC102: 74377N, Package_DIP:DIP-20_W7.62mm, F.Cu at (312.4, 263.7)
- added IC103: 74153N, Package_DIP:DIP-16_W7.62mm, F.Cu at (355.9, 149.1)
- added IC104: 74257N, Package_DIP:DIP-16_W7.62mm, F.Cu at (366.7, 149.1)
- added IC105: 74148N, Package_DIP:DIP-16_W7.62mm, F.Cu at (203.9, 171.0)
- added IC106: 74377N, Package_DIP:DIP-20_W7.62mm, F.Cu at (323.3, 263.7)
- added IC107: 7474N, Package_DIP:DIP-14_W7.62mm, F.Cu at (399.2, 102.8)
- added IC108: 7474N, Package_DIP:DIP-14_W7.62mm, F.Cu at (410.1, 102.8)
- added IC109: 74377N, Package_DIP:DIP-20_W7.62mm, F.Cu at (334.1, 263.7)
- added IC110: 74377N, Package_DIP:DIP-20_W7.62mm, F.Cu at (345.0, 263.7)
- added IC111: 74253N, Package_DIP:DIP-16_W7.62mm, F.Cu at (214.8, 171.0)
- added IC112: 74257N, Package_DIP:DIP-16_W7.62mm, F.Cu at (225.7, 171.0)
- added IC113: 74253N, Package_DIP:DIP-16_W7.62mm, F.Cu at (236.5, 171.0)
- added IC114: 74257N, Package_DIP:DIP-16_W7.62mm, F.Cu at (247.3, 171.0)
- added IC115: 7404N, Package_DIP:DIP-14_W7.62mm, F.Cu at (420.9, 102.8)
- added IC116: 74153N, Package_DIP:DIP-16_W7.62mm, F.Cu at (258.2, 171.0)
- added IC117: 74377N, Package_DIP:DIP-20_W7.62mm, F.Cu at (355.9, 263.7)
- added IC118: 74257N, Package_DIP:DIP-16_W7.62mm, F.Cu at (269.1, 171.0)
- added IC119: 7408N, Package_DIP:DIP-14_W7.62mm, F.Cu at (431.8, 102.8)
- added IC120: 74244N, Package_DIP:DIP-20_W7.62mm, F.Cu at (366.7, 263.7)
- added IC121: 74257N, Package_DIP:DIP-16_W7.62mm, F.Cu at (279.9, 171.0)
- added IC122: 74257N, Package_DIP:DIP-16_W7.62mm, F.Cu at (290.8, 171.0)
- added IC123: 74377N, Package_DIP:DIP-20_W7.62mm, F.Cu at (203.9, 290.7)
- added IC124: 74153N, Package_DIP:DIP-16_W7.62mm, F.Cu at (301.6, 171.0)
- added IC125: 74257N, Package_DIP:DIP-16_W7.62mm, F.Cu at (312.4, 171.0)
- added IC126: 7474N, Package_DIP:DIP-14_W7.62mm, F.Cu at (442.6, 102.8)
- added IC127: 74257N, Package_DIP:DIP-16_W7.62mm, F.Cu at (323.3, 171.0)
- added IC128: 74157N, Package_DIP:DIP-16_W7.62mm, F.Cu at (334.1, 171.0)
- added IC129: 74157N, Package_DIP:DIP-16_W7.62mm, F.Cu at (345.0, 171.0)
- added IC13: 74257N, Package_DIP:DIP-16_W7.62mm, F.Cu at (290.8, 83.4)
- added IC131: 74157N, Package_DIP:DIP-16_W7.62mm, F.Cu at (366.7, 171.0)
- added IC132: 74157N, Package_DIP:DIP-16_W7.62mm, F.Cu at (203.9, 192.9)
- added IC134: 74273N, Package_DIP:DIP-20_W7.62mm, F.Cu at (214.8, 290.7)
- added IC135: 74273N, Package_DIP:DIP-20_W7.62mm, F.Cu at (225.7, 290.7)
- added IC136: 74273N, Package_DIP:DIP-20_W7.62mm, F.Cu at (236.5, 290.7)
- added IC137: 7474N, Package_DIP:DIP-14_W7.62mm, F.Cu at (453.5, 102.8)
- added IC138: 7404N, Package_DIP:DIP-14_W7.62mm, F.Cu at (464.4, 102.8)
- added IC139: 7400N, Package_DIP:DIP-14_W7.62mm, F.Cu at (377.6, 122.2)
- added IC140: 58C256P, Package_DIP:DIP-28_W7.62mm, F.Cu at (-194.1, 131.7)
- added IC142: 74257N, Package_DIP:DIP-16_W7.62mm, F.Cu at (236.5, 192.9)
- added IC143: 7408N, Package_DIP:DIP-14_W7.62mm, F.Cu at (388.4, 122.2)
- added IC145: 7410N, Package_DIP:DIP-14_W7.62mm, F.Cu at (399.2, 122.2)
- added IC146: 7408N, Package_DIP:DIP-14_W7.62mm, F.Cu at (410.1, 122.2)
- added IC147: 74257N, Package_DIP:DIP-16_W7.62mm, F.Cu at (258.2, 192.9)
- added IC148: 7400N, Package_DIP:DIP-14_W7.62mm, F.Cu at (420.9, 122.2)
- added IC149: 74138N, Package_DIP:DIP-16_W7.62mm, F.Cu at (269.1, 192.9)
- added IC15: 74257N, Package_DIP:DIP-16_W7.62mm, F.Cu at (312.4, 83.4)
- added IC150: 74244N, Package_DIP:DIP-20_W7.62mm, F.Cu at (247.3, 290.7)
- added IC151: 74244N, Package_DIP:DIP-20_W7.62mm, F.Cu at (258.2, 290.7)
- added IC153: 7432N, Package_DIP:DIP-14_W7.62mm, F.Cu at (431.8, 122.2)
- added IC154: 7404N, Package_DIP:DIP-14_W7.62mm, F.Cu at (442.6, 122.2)
- added IC155: 74257N, Package_DIP:DIP-16_W7.62mm, F.Cu at (290.8, 192.9)
- added IC156: 74257N, Package_DIP:DIP-16_W7.62mm, F.Cu at (301.6, 192.9)
- added IC157: 74377N, Package_DIP:DIP-20_W7.62mm, F.Cu at (269.1, 290.7)
- added IC158: 74377N, Package_DIP:DIP-20_W7.62mm, F.Cu at (279.9, 290.7)
- added IC159: 74377N, Package_DIP:DIP-20_W7.62mm, F.Cu at (290.8, 290.7)
- added IC161: 74244N, Package_DIP:DIP-20_W7.62mm, F.Cu at (301.6, 290.7)
- added IC162: 74377N, Package_DIP:DIP-20_W7.62mm, F.Cu at (312.4, 290.7)
- added IC163: 74244N, Package_DIP:DIP-20_W7.62mm, F.Cu at (323.3, 290.7)
- added IC164: 74138N, Package_DIP:DIP-16_W7.62mm, F.Cu at (323.3, 192.9)
- added IC165: 74377N, Package_DIP:DIP-20_W7.62mm, F.Cu at (334.1, 290.7)
- added IC166: 74377N, Package_DIP:DIP-20_W7.62mm, F.Cu at (345.0, 290.7)
- added IC167: 7432N, Package_DIP:DIP-14_W7.62mm, F.Cu at (453.5, 122.2)
- added IC168: 7420N, Package_DIP:DIP-14_W7.62mm, F.Cu at (464.4, 122.2)
- added IC169: 74377N, Package_DIP:DIP-20_W7.62mm, F.Cu at (355.9, 290.7)
- added IC17: 74244N, Package_DIP:DIP-20_W7.62mm, F.Cu at (236.5, 236.7)
- added IC170: 74253N, Package_DIP:DIP-16_W7.62mm, F.Cu at (334.1, 192.9)
- added IC171: 74377N, Package_DIP:DIP-20_W7.62mm, F.Cu at (366.7, 290.7)
- added IC172: 74377N, Package_DIP:DIP-20_W7.62mm, F.Cu at (203.9, 317.7)
- added IC173: 7427N, Package_DIP:DIP-14_W7.62mm, F.Cu at (377.6, 141.6)
- added IC174: 7432N, Package_DIP:DIP-14_W7.62mm, F.Cu at (388.4, 141.6)
- added IC175: 7486N, Package_DIP:DIP-14_W7.62mm, F.Cu at (399.2, 141.6)
- added IC176: 7404N, Package_DIP:DIP-14_W7.62mm, F.Cu at (410.1, 141.6)
- added IC177: 74377N, Package_DIP:DIP-20_W7.62mm, F.Cu at (214.8, 317.7)
- added IC178: 74377N, Package_DIP:DIP-20_W7.62mm, F.Cu at (225.7, 317.7)
- added IC179: 74253N, Package_DIP:DIP-16_W7.62mm, F.Cu at (345.0, 192.9)
- added IC18: 7432N, Package_DIP:DIP-14_W7.62mm, F.Cu at (377.6, 83.4)
- added IC180: 74153N, Package_DIP:DIP-16_W7.62mm, F.Cu at (355.9, 192.9)
- added IC181: 74253N, Package_DIP:DIP-16_W7.62mm, F.Cu at (366.7, 192.9)
- added IC182: 74253N, Package_DIP:DIP-16_W7.62mm, F.Cu at (203.9, 214.8)
- added IC183: 74377N, Package_DIP:DIP-20_W7.62mm, F.Cu at (236.5, 317.7)
- added IC184: 74377N, Package_DIP:DIP-20_W7.62mm, F.Cu at (247.3, 317.7)
- added IC185: 74244N, Package_DIP:DIP-20_W7.62mm, F.Cu at (258.2, 317.7)
- added IC189: 74244N, Package_DIP:DIP-20_W7.62mm, F.Cu at (269.1, 317.7)
- added IC19: 74377N, Package_DIP:DIP-20_W7.62mm, F.Cu at (247.3, 236.7)
- added IC190: 7474N, Package_DIP:DIP-14_W7.62mm, F.Cu at (420.9, 141.6)
- added IC191: 74244N, Package_DIP:DIP-20_W7.62mm, F.Cu at (279.9, 317.7)
- added IC192: 74279N, Package_DIP:DIP-16_W7.62mm, F.Cu at (214.8, 214.8)
- added IC193: 74279N, Package_DIP:DIP-16_W7.62mm, F.Cu at (225.7, 214.8)
- added IC194: 74279N, Package_DIP:DIP-16_W7.62mm, F.Cu at (236.5, 214.8)
- added IC195: 74244N, Package_DIP:DIP-20_W7.62mm, F.Cu at (290.8, 317.7)
- added IC196: 7404N, Package_DIP:DIP-14_W7.62mm, F.Cu at (431.8, 141.6)
- added IC197: 74244N, Package_DIP:DIP-20_W7.62mm, F.Cu at (301.6, 317.7)
- added IC198: 74244N, Package_DIP:DIP-20_W7.62mm, F.Cu at (312.4, 317.7)
- added IC200: 74244N, Package_DIP:DIP-20_W7.62mm, F.Cu at (323.3, 317.7)
- added IC201: 7408N, Package_DIP:DIP-14_W7.62mm, F.Cu at (442.6, 141.6)
- added IC202: 7427N, Package_DIP:DIP-14_W7.62mm, F.Cu at (453.5, 141.6)
- added IC203: 7430N, Package_DIP:DIP-14_W7.62mm, F.Cu at (464.4, 141.6)
- added IC204: 74377N, Package_DIP:DIP-20_W7.62mm, F.Cu at (334.1, 317.7)
- added IC205: 7404N, Package_DIP:DIP-14_W7.62mm, F.Cu at (377.6, 161.0)
- added IC206: 74257N, Package_DIP:DIP-16_W7.62mm, F.Cu at (247.3, 214.8)
- added IC207: 74244N, Package_DIP:DIP-20_W7.62mm, F.Cu at (345.0, 317.7)
- added IC208: 74245N, Package_DIP:DIP-20_W7.62mm, F.Cu at (355.9, 317.7)
- added IC209: 74244N, Package_DIP:DIP-20_W7.62mm, F.Cu at (366.7, 317.7)
- added IC21: 58C256P, Package_DIP:DIP-28_W7.62mm, F.Cu at (-204.9, 131.7)
- added IC210: 74377N, Package_DIP:DIP-20_W7.62mm, F.Cu at (203.9, 344.7)
- added IC211: 74244N, Package_DIP:DIP-20_W7.62mm, F.Cu at (214.8, 344.7)
- added IC212: 74244N, Package_DIP:DIP-20_W7.62mm, F.Cu at (225.7, 344.7)
- added IC213: 74244N, Package_DIP:DIP-20_W7.62mm, F.Cu at (236.5, 344.7)
- added IC214: 74138N, Package_DIP:DIP-16_W7.62mm, F.Cu at (258.2, 214.8)
- added IC22: 7408N, Package_DIP:DIP-14_W7.62mm, F.Cu at (388.4, 83.4)
- added IC231: 74273N, Package_DIP:DIP-20_W7.62mm, F.Cu at (247.3, 344.7)
- added IC236: 7408N, Package_DIP:DIP-14_W7.62mm, F.Cu at (388.4, 161.0)
- added IC237: 74153N, Package_DIP:DIP-16_W7.62mm, F.Cu at (269.1, 214.8)
- added IC24: 74157N, Package_DIP:DIP-16_W7.62mm, F.Cu at (355.9, 83.4)
- added IC241: 74153N, Package_DIP:DIP-16_W7.62mm, F.Cu at (279.9, 214.8)
- added IC245: 74377N, Package_DIP:DIP-20_W7.62mm, F.Cu at (258.2, 344.7)
- added IC25: 7427N, Package_DIP:DIP-14_W7.62mm, F.Cu at (399.2, 83.4)
- added IC255: 74153N, Package_DIP:DIP-16_W7.62mm, F.Cu at (290.8, 214.8)
- added IC259: 74273N, Package_DIP:DIP-20_W7.62mm, F.Cu at (269.1, 344.7)
- added IC26: 74244N, Package_DIP:DIP-20_W7.62mm, F.Cu at (258.2, 236.7)
- added IC260: 74377N, Package_DIP:DIP-20_W7.62mm, F.Cu at (279.9, 344.7)
- added IC263: 7432N, Package_DIP:DIP-14_W7.62mm, F.Cu at (399.2, 161.0)
- added IC266: 74273N, Package_DIP:DIP-20_W7.62mm, F.Cu at (290.8, 344.7)
- added IC267: 74273N, Package_DIP:DIP-20_W7.62mm, F.Cu at (301.6, 344.7)
- added IC27: 74244N, Package_DIP:DIP-20_W7.62mm, F.Cu at (269.1, 236.7)
- added IC270: 74153N, Package_DIP:DIP-16_W7.62mm, F.Cu at (301.6, 214.8)
- added IC28: 74377N, Package_DIP:DIP-20_W7.62mm, F.Cu at (279.9, 236.7)
- added IC29: 74153N, Package_DIP:DIP-16_W7.62mm, F.Cu at (366.7, 83.4)
- added IC30: 74151N, Package_DIP:DIP-16_W7.62mm, F.Cu at (203.9, 105.3)
- added IC31: 74377N, Package_DIP:DIP-20_W7.62mm, F.Cu at (290.8, 236.7)
- added IC32: 74273N, Package_DIP:DIP-20_W7.62mm, F.Cu at (301.6, 236.7)
- added IC33: 74273N, Package_DIP:DIP-20_W7.62mm, F.Cu at (312.4, 236.7)
- added IC334: 74273N, Package_DIP:DIP-20_W7.62mm, F.Cu at (312.4, 344.7)
- added IC336: 74273N, Package_DIP:DIP-20_W7.62mm, F.Cu at (323.3, 344.7)
- added IC338: 74273N, Package_DIP:DIP-20_W7.62mm, F.Cu at (334.1, 344.7)
- added IC34: 74153N, Package_DIP:DIP-16_W7.62mm, F.Cu at (214.8, 105.3)
- added IC341: 74257N, Package_DIP:DIP-16_W7.62mm, F.Cu at (312.4, 214.8)
- added IC35: 74153N, Package_DIP:DIP-16_W7.62mm, F.Cu at (225.7, 105.3)
- added IC36: 74153N, Package_DIP:DIP-16_W7.62mm, F.Cu at (236.5, 105.3)
- added IC37: 74153N, Package_DIP:DIP-16_W7.62mm, F.Cu at (247.3, 105.3)
- added IC38: 74153N, Package_DIP:DIP-16_W7.62mm, F.Cu at (258.2, 105.3)
- added IC39: 74257N, Package_DIP:DIP-16_W7.62mm, F.Cu at (269.1, 105.3)
- added IC4: 74244N, Package_DIP:DIP-20_W7.62mm, F.Cu at (214.8, 236.7)
- added IC40: 74153N, Package_DIP:DIP-16_W7.62mm, F.Cu at (279.9, 105.3)
- added IC41: 74151N, Package_DIP:DIP-16_W7.62mm, F.Cu at (290.8, 105.3)
- added IC411: 74279N, Package_DIP:DIP-16_W7.62mm, F.Cu at (323.3, 214.8)
- added IC412: 74173N, Package_DIP:DIP-16_W7.62mm, F.Cu at (334.1, 214.8)
- added IC43: 7404N, Package_DIP:DIP-14_W7.62mm, F.Cu at (410.1, 83.4)
- added IC45: 7408N, Package_DIP:DIP-14_W7.62mm, F.Cu at (420.9, 83.4)
- added IC46: 74283N, Package_DIP:DIP-16_W7.62mm, F.Cu at (323.3, 105.3)
- added IC47: 74153N, Package_DIP:DIP-16_W7.62mm, F.Cu at (334.1, 105.3)
- added IC48: 74377N, Package_DIP:DIP-20_W7.62mm, F.Cu at (323.3, 236.7)
- added IC49: 74257N, Package_DIP:DIP-16_W7.62mm, F.Cu at (345.0, 105.3)
- added IC50: 74283N, Package_DIP:DIP-16_W7.62mm, F.Cu at (355.9, 105.3)
- added IC51: 74283N, Package_DIP:DIP-16_W7.62mm, F.Cu at (366.7, 105.3)
- added IC52: 74283N, Package_DIP:DIP-16_W7.62mm, F.Cu at (203.9, 127.2)
- added IC54: 74157N, Package_DIP:DIP-16_W7.62mm, F.Cu at (225.7, 127.2)
- added IC55: 74257N, Package_DIP:DIP-16_W7.62mm, F.Cu at (236.5, 127.2)
- added IC57: 74377N, Package_DIP:DIP-20_W7.62mm, F.Cu at (334.1, 236.7)
- added IC58: 7411N, Package_DIP:DIP-14_W7.62mm, F.Cu at (431.8, 83.4)
- added IC59: 7486N, Package_DIP:DIP-14_W7.62mm, F.Cu at (442.6, 83.4)
- added IC60: 74273N, Package_DIP:DIP-20_W7.62mm, F.Cu at (345.0, 236.7)
- added IC63: 74257N, Package_DIP:DIP-16_W7.62mm, F.Cu at (279.9, 127.2)
- added IC64: 74153N, Package_DIP:DIP-16_W7.62mm, F.Cu at (290.8, 127.2)
- added IC65: 74244N, Package_DIP:DIP-20_W7.62mm, F.Cu at (355.9, 236.7)
- added IC66: 74377N, Package_DIP:DIP-20_W7.62mm, F.Cu at (366.7, 236.7)
- added IC7: 74157N, Package_DIP:DIP-16_W7.62mm, F.Cu at (258.2, 83.4)
- added IC70: 7404N, Package_DIP:DIP-14_W7.62mm, F.Cu at (453.5, 83.4)
- added IC72: 74244N, Package_DIP:DIP-20_W7.62mm, F.Cu at (203.9, 263.7)
- added IC73: 74153N, Package_DIP:DIP-16_W7.62mm, F.Cu at (345.0, 127.2)
- added IC74: 7474N, Package_DIP:DIP-14_W7.62mm, F.Cu at (464.4, 83.4)
- added IC75: 74273N, Package_DIP:DIP-20_W7.62mm, F.Cu at (214.8, 263.7)
- added IC76: 74273N, Package_DIP:DIP-20_W7.62mm, F.Cu at (225.7, 263.7)
- added IC77: 74273N, Package_DIP:DIP-20_W7.62mm, F.Cu at (236.5, 263.7)
- added IC78: 74273N, Package_DIP:DIP-20_W7.62mm, F.Cu at (247.3, 263.7)
- added IC79: 74273N, Package_DIP:DIP-20_W7.62mm, F.Cu at (258.2, 263.7)
- added IC8: 74377N, Package_DIP:DIP-20_W7.62mm, F.Cu at (225.7, 236.7)
- added IC83: 74153N, Package_DIP:DIP-16_W7.62mm, F.Cu at (214.8, 149.1)
- added IC90: 74377N, Package_DIP:DIP-20_W7.62mm, F.Cu at (269.1, 263.7)
- added IC91: 74253N, Package_DIP:DIP-16_W7.62mm, F.Cu at (290.8, 149.1)
- added IC92: 74153N, Package_DIP:DIP-16_W7.62mm, F.Cu at (301.6, 149.1)
- added IC93: 7408N, Package_DIP:DIP-14_W7.62mm, F.Cu at (377.6, 102.8)
- added IC94: 7432N, Package_DIP:DIP-14_W7.62mm, F.Cu at (388.4, 102.8)
- added IC95: 74253N, Package_DIP:DIP-16_W7.62mm, F.Cu at (312.4, 149.1)
- added IC96: 74157N, Package_DIP:DIP-16_W7.62mm, F.Cu at (323.3, 149.1)
- added IC97: 74244N, Package_DIP:DIP-20_W7.62mm, F.Cu at (279.9, 263.7)
- added IC98: 74257N, Package_DIP:DIP-16_W7.62mm, F.Cu at (334.1, 149.1)
- added IC99: 74377N, Package_DIP:DIP-20_W7.62mm, F.Cu at (290.8, 263.7)
- added IC_02_0: 7402N, Package_DIP:DIP-14_W7.62mm, F.Cu at (410.1, 161.0)
- added IC_04_2: 7404N, Package_DIP:DIP-14_W7.62mm, F.Cu at (420.9, 161.0)
- added IC_10_0: 7410N, Package_DIP:DIP-14_W7.62mm, F.Cu at (431.8, 161.0)
- added IC_86_0: 7486N, Package_DIP:DIP-14_W7.62mm, F.Cu at (442.6, 161.0)
- added IC_86_1: 7486N, Package_DIP:DIP-14_W7.62mm, F.Cu at (453.5, 161.0)
- added INT_CODE_REG1: 74377N, Package_DIP:DIP-20_W7.62mm, F.Cu at (345.0, 344.7)
- added INT_STATUS_REG0: 74273N, Package_DIP:DIP-20_W7.62mm, F.Cu at (355.9, 344.7)
- added SW1: SW_DIP-8, Button_Switch_THT:SW_DIP_SPSTx08_Slide_6.7x21.88mm_W7.62mm_P2.54mm_LowProfile, F.Cu at (487.7, 378.8)
- added SW2: SW_DIP-8, Button_Switch_THT:SW_DIP_SPSTx08_Slide_6.7x21.88mm_W7.62mm_P2.54mm_LowProfile, F.Cu at (498.5, 378.8)
- added SW3: SW_DIP-8, Button_Switch_THT:SW_DIP_SPSTx08_Slide_6.7x21.88mm_W7.62mm_P2.54mm_LowProfile, F.Cu at (509.4, 378.8)
- added SW4: SW_DIP-8, Button_Switch_THT:SW_DIP_SPSTx08_Slide_6.7x21.88mm_W7.62mm_P2.54mm_LowProfile, F.Cu at (520.2, 378.8)
- added SW5: SW_DIP-8, Button_Switch_THT:SW_DIP_SPSTx08_Slide_6.7x21.88mm_W7.62mm_P2.54mm_LowProfile, F.Cu at (531.1, 378.8)
- added SW6: SW_DIP-8, Button_Switch_THT:SW_DIP_SPSTx08_Slide_6.7x21.88mm_W7.62mm_P2.54mm_LowProfile, F.Cu at (541.9, 378.8)
- added SW7: SW_DIP-8, Button_Switch_THT:SW_DIP_SPSTx08_Slide_6.7x21.88mm_W7.62mm_P2.54mm_LowProfile, F.Cu at (552.8, 378.8)
- added SW8: SW_DIP-8, Button_Switch_THT:SW_DIP_SPSTx08_Slide_6.7x21.88mm_W7.62mm_P2.54mm_LowProfile, F.Cu at (563.6, 378.8)
- added SW9: SW_DIP-8, Button_Switch_THT:SW_DIP_SPSTx08_Slide_6.7x21.88mm_W7.62mm_P2.54mm_LowProfile, F.Cu at (574.5, 378.8)
- added U1: as6c4008-55pcn, Package_DIP:DIP-32_W15.24mm, F.Cu at (-352.2, 131.7)
- added U10: 16550, Package_DIP:DIP-40_W15.24mm, F.Cu at (-344.8, 16.8)
- added U11: 16550, Package_DIP:DIP-40_W15.24mm, F.Cu at (-326.4, 16.8)
- added U12: 8253, Package_DIP:DIP-24_W15.24mm, F.Cu at (-252.8, 16.8)
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Other:
- board outline added: 1066 x 710 mm

Commit message: kicad
Parts:
- removed BIOS_RAM1: 431000, Package_DIP:DIP-32_W15.24mm
- removed FLAGS0, IC231, IC259, IC266, IC267, IC334, IC336, IC338, INT_STATUS_REG0: 74273N, Package_DIP:DIP-20_W7.62mm
- removed IC209, IC211, IC212, IC213: 74244N, Package_DIP:DIP-20_W7.62mm
- removed IC210, IC245, IC260, INT_CODE_REG1: 74377N, Package_DIP:DIP-20_W7.62mm
- removed IC214: 74138N, Package_DIP:DIP-16_W7.62mm
- removed IC236: 7408N, Package_DIP:DIP-14_W7.62mm
- removed IC237, IC241, IC255, IC270: 74153N, Package_DIP:DIP-16_W7.62mm
- removed IC263: 7432N, Package_DIP:DIP-14_W7.62mm
- removed IC341: 74257N, Package_DIP:DIP-16_W7.62mm
- removed IC411: 74279N, Package_DIP:DIP-16_W7.62mm
- removed IC412: 74173N, Package_DIP:DIP-16_W7.62mm
- removed IC_02_0: 7402N, Package_DIP:DIP-14_W7.62mm
- removed IC_04_2: 7404N, Package_DIP:DIP-14_W7.62mm
- removed IC_10_0: 7410N, Package_DIP:DIP-14_W7.62mm
- removed IC_86_0: 7486N, Package_DIP:DIP-14_W7.62mm
- removed U_ROM0: 27512, Package_DIP:DIP-28_W15.24mm
- added FLAGS1: 74273N, Package_DIP:DIP-20_W7.62mm, F.Cu at (-2.80, 93.9)
- added IC10: 74153N, Package_DIP:DIP-16_W7.62mm, F.Cu at (73.2, -81.3)
- added IC11: 74257N, Package_DIP:DIP-16_W7.62mm, F.Cu at (84.0, -81.3)
- added IC186: 74244N, Package_DIP:DIP-20_W7.62mm, F.Cu at (127.4, 174.9)
- added IC187: 74279N, Package_DIP:DIP-16_W7.62mm, F.Cu at (138.2, 28.2)
- added IC188: 74279N, Package_DIP:DIP-16_W7.62mm, F.Cu at (149.1, 28.2)
- added IC199: 74244N, Package_DIP:DIP-20_W7.62mm, F.Cu at (8.05, 201.9)
- added IC_02_1: 7402N, Package_DIP:DIP-14_W7.62mm, F.Cu at (192.5, -23.1)
- added IC_04_1: 7404N, Package_DIP:DIP-14_W7.62mm, F.Cu at (203.3, -23.1)
- added IC_10_1: 7410N, Package_DIP:DIP-14_W7.62mm, F.Cu at (214.2, -23.1)
- added IC_86_2: 7486N, Package_DIP:DIP-14_W7.62mm, F.Cu at (235.9, -23.1)
- added IRQ_0_DFF1: 7474N, Package_DIP:DIP-14_W7.62mm, F.Cu at (246.8, -23.1)
- added IRQ_1_DFF1: 7474N, Package_DIP:DIP-14_W7.62mm, F.Cu at (257.6, -23.1)
- added IRQ_2_DFF1: 7474N, Package_DIP:DIP-14_W7.62mm, F.Cu at (268.4, -23.1)
- added IRQ_3_DFF1: 7474N, Package_DIP:DIP-14_W7.62mm, F.Cu at (279.3, -23.1)
- added IRQ_4_DFF1: 7474N, Package_DIP:DIP-14_W7.62mm, F.Cu at (181.7, -3.66)
- added IRQ_5_DFF1: 7474N, Package_DIP:DIP-14_W7.62mm, F.Cu at (192.5, -3.66)
- added IRQ_6_DFF1: 7474N, Package_DIP:DIP-14_W7.62mm, F.Cu at (203.3, -3.66)
- added IRQ_7_DFF1: 7474N, Package_DIP:DIP-14_W7.62mm, F.Cu at (214.2, -3.66)
- added IRQ_AND_1: 7408N, Package_DIP:DIP-14_W7.62mm, F.Cu at (225.1, -3.66)
- added IRQ_AND_2: 7408N, Package_DIP:DIP-14_W7.62mm, F.Cu at (235.9, -3.66)
- added IRQ_CODE1: 74377N, Package_DIP:DIP-20_W7.62mm, F.Cu at (94.8, 201.9)
- added IRQ_ENCODER1: 74148N, Package_DIP:DIP-16_W7.62mm, F.Cu at (8.05, 50.1)
- added IRQ_RST_DECODER1: 74138N, Package_DIP:DIP-16_W7.62mm, F.Cu at (18.9, 50.1)
- added IRQ_STATUS_1: 74273N, Package_DIP:DIP-20_W7.62mm, F.Cu at (105.7, 201.9)
- added MARH1: 74377N, Package_DIP:DIP-20_W7.62mm, F.Cu at (116.5, 201.9)
- added MARL1: 74377N, Package_DIP:DIP-20_W7.62mm, F.Cu at (127.4, 201.9)
- added MDRH1: 74377N, Package_DIP:DIP-20_W7.62mm, F.Cu at (138.2, 201.9)
- added MDRL1: 74377N, Package_DIP:DIP-20_W7.62mm, F.Cu at (149.1, 201.9)
- added MDR_IN_MUX_1: 74157N, Package_DIP:DIP-16_W7.62mm, F.Cu at (29.8, 50.1)
- added MDR_IN_MUX_2: 74157N, Package_DIP:DIP-16_W7.62mm, F.Cu at (40.6, 50.1)
- added MDR_OUT_MUX_1: 74157N, Package_DIP:DIP-16_W7.62mm, F.Cu at (51.5, 50.1)
- added MDR_OUT_MUX_2: 74157N, Package_DIP:DIP-16_W7.62mm, F.Cu at (62.3, 50.1)
- added RN1: R_Pack08, Package_DIP:DIP-16_W7.62mm, F.Cu at (73.2, 50.1)
- added RN2: R_Pack08, Package_DIP:DIP-16_W7.62mm, F.Cu at (84.0, 50.1)
- added RN3: R_Pack08, Package_DIP:DIP-16_W7.62mm, F.Cu at (94.8, 50.1)
- added RN4: R_Pack08, Package_DIP:DIP-16_W7.62mm, F.Cu at (105.7, 50.1)
- added RN5: R_Pack08, Package_DIP:DIP-16_W7.62mm, F.Cu at (116.5, 50.1)
- added RN6: R_Pack08, Package_DIP:DIP-16_W7.62mm, F.Cu at (127.4, 50.1)
- added RN7: R_Pack08, Package_DIP:DIP-16_W7.62mm, F.Cu at (138.2, 50.1)
- added RN8: R_Pack08, Package_DIP:DIP-16_W7.62mm, F.Cu at (149.1, 50.1)
- added RN9: R_Pack08, Package_DIP:DIP-16_W7.62mm, F.Cu at (159.9, 50.1)
- added SW10: SW_DIP_x08, Package_DIP:DIP-16_W7.62mm, F.Cu at (84.0, 72.0)
- added U16: 4040, Package_DIP:DIP-16_W7.62mm, F.Cu at (94.8, 72.0)
- added U_ROM15: 27512, Package_DIP:DIP-28_W15.24mm, F.Cu at (-268.6, -29.0)
- IC1, IC114, IC55, IC63: value 74257N -> 74377N; footprint Package_DIP:DIP-16_W7.62mm -> Package_DIP:DIP-20_W7.62mm
- IC100, IC104, IC98: value 74257N -> 74273N; footprint Package_DIP:DIP-16_W7.62mm -> Package_DIP:DIP-20_W7.62mm
- IC101, IC102, IC106, IC99: value 74377N -> 74273N
- IC103, IC92: value 74153N -> 74273N; footprint Package_DIP:DIP-16_W7.62mm -> Package_DIP:DIP-20_W7.62mm
- IC105: value 74148N -> 74273N; footprint Package_DIP:DIP-16_W7.62mm -> Package_DIP:DIP-20_W7.62mm
- IC107, IC108: value 7474N -> 74273N; footprint Package_DIP:DIP-14_W7.62mm -> Package_DIP:DIP-20_W7.62mm
- IC109, IC165: value 74377N -> 7427N; footprint Package_DIP:DIP-20_W7.62mm -> Package_DIP:DIP-14_W7.62mm
- IC110: value 74377N -> 74245N
- IC111: value 74253N -> 74257N
- IC113: value 74253N -> 7404N; footprint Package_DIP:DIP-16_W7.62mm -> Package_DIP:DIP-14_W7.62mm
- IC115, IC196, IC205: value 7404N -> 74244N; footprint Package_DIP:DIP-14_W7.62mm -> Package_DIP:DIP-20_W7.62mm
- IC116: value 74153N -> 74138N
- IC117, IC172, IC204: value 74377N -> 74244N
- IC118, IC206: value 74257N -> 74244N; footprint Package_DIP:DIP-16_W7.62mm -> Package_DIP:DIP-20_W7.62mm
- IC119, IC201: value 7408N -> 74244N; footprint Package_DIP:DIP-14_W7.62mm -> Package_DIP:DIP-20_W7.62mm
- IC12, IC16, IC160, IC20, IC30: value 74151N -> 74257N
- IC121: value 74257N -> 7404N; footprint Package_DIP:DIP-16_W7.62mm -> Package_DIP:DIP-14_W7.62mm
- IC122: value 74257N -> 7420N; footprint Package_DIP:DIP-16_W7.62mm -> Package_DIP:DIP-14_W7.62mm
- IC123, IC28, IC90: value 74377N -> 74151N; footprint Package_DIP:DIP-20_W7.62mm -> Package_DIP:DIP-16_W7.62mm
- IC124: value 74153N -> 74151N
- IC125, IC127, IC142, IC147, IC49: value 74257N -> 74151N
- IC126, IC137: value 7474N -> 74151N; footprint Package_DIP:DIP-14_W7.62mm -> Package_DIP:DIP-16_W7.62mm
- IC128, IC129, IC131, IC132: value 74157N -> 74151N
- IC13: value 74257N -> 7408N; footprint Package_DIP:DIP-16_W7.62mm -> Package_DIP:DIP-14_W7.62mm
- IC134, IC135, IC136: value 74273N -> 74151N; footprint Package_DIP:DIP-20_W7.62mm -> Package_DIP:DIP-16_W7.62mm
- IC138, IC154: value 7404N -> 74151N; footprint Package_DIP:DIP-14_W7.62mm -> Package_DIP:DIP-16_W7.62mm
- IC139, IC148: value 7400N -> 74151N; footprint Package_DIP:DIP-14_W7.62mm -> Package_DIP:DIP-16_W7.62mm
- IC14, IC80, IC81, IC82, IC87, IC89, IC9: value 74151N -> 74153N
- IC140: value 58C256P -> 74151N; footprint Package_DIP:DIP-28_W7.62mm -> Package_DIP:DIP-16_W7.62mm
- IC143, IC146: value 7408N -> 74151N; footprint Package_DIP:DIP-14_W7.62mm -> Package_DIP:DIP-16_W7.62mm
- IC145: value 7410N -> 74151N; footprint Package_DIP:DIP-14_W7.62mm -> Package_DIP:DIP-16_W7.62mm
- IC149: value 74138N -> 74151N
- IC150, IC151: value 74244N -> 74151N; footprint Package_DIP:DIP-20_W7.62mm -> Package_DIP:DIP-16_W7.62mm
- IC153: value 7432N -> 74151N; footprint Package_DIP:DIP-14_W7.62mm -> Package_DIP:DIP-16_W7.62mm
- IC157, IC158, IC159, IC19: value 74377N -> 74257N; footprint Package_DIP:DIP-20_W7.62mm -> Package_DIP:DIP-16_W7.62mm
- IC161: value 74244N -> 7408N; footprint Package_DIP:DIP-20_W7.62mm -> Package_DIP:DIP-14_W7.62mm
- IC162: value 74377N -> 7430N; footprint Package_DIP:DIP-20_W7.62mm -> Package_DIP:DIP-14_W7.62mm
- IC163: value 74244N -> 7404N; footprint Package_DIP:DIP-20_W7.62mm -> Package_DIP:DIP-14_W7.62mm
- IC164: value 74138N -> 7474N; footprint Package_DIP:DIP-16_W7.62mm -> Package_DIP:DIP-14_W7.62mm
- IC166, IC169, IC8: value 74377N -> 74153N; footprint Package_DIP:DIP-20_W7.62mm -> Package_DIP:DIP-16_W7.62mm
- IC167, IC18: value 7432N -> 74153N; footprint Package_DIP:DIP-14_W7.62mm -> Package_DIP:DIP-16_W7.62mm
- IC168: value 7420N -> 74153N; footprint Package_DIP:DIP-14_W7.62mm -> Package_DIP:DIP-16_W7.62mm
- IC17: value 74244N -> 74153N; footprint Package_DIP:DIP-20_W7.62mm -> Package_DIP:DIP-16_W7.62mm
- IC170: value 74253N -> 7474N; footprint Package_DIP:DIP-16_W7.62mm -> Package_DIP:DIP-14_W7.62mm
- IC171: value 74377N -> 74173N; footprint Package_DIP:DIP-20_W7.62mm -> Package_DIP:DIP-16_W7.62mm
- IC173, IC202: value 7427N -> 74244N; footprint Package_DIP:DIP-14_W7.62mm -> Package_DIP:DIP-20_W7.62mm
- IC174: value 7432N -> 74244N; footprint Package_DIP:DIP-14_W7.62mm -> Package_DIP:DIP-20_W7.62mm
- IC175: value 7486N -> 74279N; footprint Package_DIP:DIP-14_W7.62mm -> Package_DIP:DIP-16_W7.62mm
- IC176: value 7404N -> 74138N; footprint Package_DIP:DIP-14_W7.62mm -> Package_DIP:DIP-16_W7.62mm
- IC177, IC178: value 74377N -> 58C256P; footprint Package_DIP:DIP-20_W7.62mm -> Package_DIP:DIP-28_W7.62mm
- IC179: value 74253N -> 74244N; footprint Package_DIP:DIP-16_W7.62mm -> Package_DIP:DIP-20_W7.62mm
- IC180, IC47: value 74153N -> 74244N; footprint Package_DIP:DIP-16_W7.62mm -> Package_DIP:DIP-20_W7.62mm
- IC181, IC182: value 74253N -> 74157N
- IC183, IC184: value 74377N -> 74157N; footprint Package_DIP:DIP-20_W7.62mm -> Package_DIP:DIP-16_W7.62mm
- IC189: value 74244N -> 74279N; footprint Package_DIP:DIP-20_W7.62mm -> Package_DIP:DIP-16_W7.62mm
- IC190: value 7474N -> 74257N; footprint Package_DIP:DIP-14_W7.62mm -> Package_DIP:DIP-16_W7.62mm
- IC191, IC26, IC27: value 74244N -> 74257N; footprint Package_DIP:DIP-20_W7.62mm -> Package_DIP:DIP-16_W7.62mm
- IC192: value 74279N -> 7432N; footprint Package_DIP:DIP-16_W7.62mm -> Package_DIP:DIP-14_W7.62mm
- IC193, IC194: value 74279N -> 7404N; footprint Package_DIP:DIP-16_W7.62mm -> Package_DIP:DIP-14_W7.62mm
- IC195, IC65, IC72: value 74244N -> 74377N
- IC2, IC42, IC56, IC61, IC62, IC67, IC68, IC69, IC71, IC84, IC85: value 74151N -> 74377N; footprint Package_DIP:DIP-16_W7.62mm -> Package_DIP:DIP-20_W7.62mm
- IC203: value 7430N -> 74244N; footprint Package_DIP:DIP-14_W7.62mm -> Package_DIP:DIP-20_W7.62mm
- IC207: value 74244N -> 7400N; footprint Package_DIP:DIP-20_W7.62mm -> Package_DIP:DIP-14_W7.62mm
- IC208: value 74245N -> 7400N; footprint Package_DIP:DIP-20_W7.62mm -> Package_DIP:DIP-14_W7.62mm
- IC21: value 58C256P -> 7404N; footprint Package_DIP:DIP-28_W7.62mm -> Package_DIP:DIP-14_W7.62mm
- IC22: value 7408N -> 74273N; footprint Package_DIP:DIP-14_W7.62mm -> Package_DIP:DIP-20_W7.62mm
- IC23: value 74151N -> 7410N; footprint Package_DIP:DIP-16_W7.62mm -> Package_DIP:DIP-14_W7.62mm
- IC24: value 74157N -> 74257N
- IC25: value 7427N -> 74257N; footprint Package_DIP:DIP-14_W7.62mm -> Package_DIP:DIP-16_W7.62mm
- IC29: value 74153N -> 7432N; footprint Package_DIP:DIP-16_W7.62mm -> Package_DIP:DIP-14_W7.62mm
- IC3, IC5, IC6: value 74151N -> 74253N
- IC31: value 74377N -> 74253N; footprint Package_DIP:DIP-20_W7.62mm -> Package_DIP:DIP-16_W7.62mm
- IC32, IC33: value 74273N -> 74253N; footprint Package_DIP:DIP-20_W7.62mm -> Package_DIP:DIP-16_W7.62mm
- IC34: value 74153N -> 74253N
- IC35: value 74153N -> 7408N; footprint Package_DIP:DIP-16_W7.62mm -> Package_DIP:DIP-14_W7.62mm
- IC36, IC64, IC73: value 74153N -> 74377N; footprint Package_DIP:DIP-16_W7.62mm -> Package_DIP:DIP-20_W7.62mm
- IC37: value 74153N -> 7486N; footprint Package_DIP:DIP-16_W7.62mm -> Package_DIP:DIP-14_W7.62mm
- IC38, IC40: value 74153N -> 74283N
- IC39: value 74257N -> 74283N
- IC4: value 74244N -> 74253N; footprint Package_DIP:DIP-20_W7.62mm -> Package_DIP:DIP-16_W7.62mm
- IC41: value 74151N -> 74283N
- IC43: value 7404N -> 7408N
- IC44, IC53: value 74151N -> 7432N; footprint Package_DIP:DIP-16_W7.62mm -> Package_DIP:DIP-14_W7.62mm
- IC45: value 7408N -> 7432N
- IC46, IC52: value 74283N -> 7408N; footprint Package_DIP:DIP-16_W7.62mm -> Package_DIP:DIP-14_W7.62mm
- IC48: value 74377N -> 7432N; footprint Package_DIP:DIP-20_W7.62mm -> Package_DIP:DIP-14_W7.62mm
- IC50: value 74283N -> 74151N
- IC51: value 74283N -> 7427N; footprint Package_DIP:DIP-16_W7.62mm -> Package_DIP:DIP-14_W7.62mm
- IC54: value 74157N -> 74377N; footprint Package_DIP:DIP-16_W7.62mm -> Package_DIP:DIP-20_W7.62mm
- IC58: value 7411N -> 74377N; footprint Package_DIP:DIP-14_W7.62mm -> Package_DIP:DIP-20_W7.62mm
- IC59: value 7486N -> 74377N; footprint Package_DIP:DIP-14_W7.62mm -> Package_DIP:DIP-20_W7.62mm
- IC60: value 74273N -> 74377N
- IC7: value 74157N -> 74153N
- IC70: value 7404N -> 74377N; footprint Package_DIP:DIP-14_W7.62mm -> Package_DIP:DIP-20_W7.62mm
- IC74: value 7474N -> 74377N; footprint Package_DIP:DIP-14_W7.62mm -> Package_DIP:DIP-20_W7.62mm
- IC75: value 74273N -> 7411N; footprint Package_DIP:DIP-20_W7.62mm -> Package_DIP:DIP-14_W7.62mm
- IC76: value 74273N -> 74257N; footprint Package_DIP:DIP-20_W7.62mm -> Package_DIP:DIP-16_W7.62mm
- IC77, IC78, IC79: value 74273N -> 74153N; footprint Package_DIP:DIP-20_W7.62mm -> Package_DIP:DIP-16_W7.62mm
- IC86: value 74151N -> 7486N; footprint Package_DIP:DIP-16_W7.62mm -> Package_DIP:DIP-14_W7.62mm
- IC91, IC95: value 74253N -> 74273N; footprint Package_DIP:DIP-16_W7.62mm -> Package_DIP:DIP-20_W7.62mm
- IC93: value 7408N -> 74257N; footprint Package_DIP:DIP-14_W7.62mm -> Package_DIP:DIP-16_W7.62mm
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Connections:
- BIOS_ROM1 pad 10: Net-(BIOS_RAM1-A0) -> Net-(BIOS_ROM1A-A0)
- BIOS_ROM1 pad 11: Net-(BIOS_RAM1-I/O1) -> Net-(BIOS_ROM1A-O0)
- BIOS_ROM1 pad 12: Net-(BIOS_RAM1-I/O2) -> Net-(BIOS_ROM1A-O1)
- BIOS_ROM1 pad 13: Net-(BIOS_RAM1-I/O3) -> Net-(BIOS_ROM1A-O2)
- BIOS_ROM1 pad 15: Net-(BIOS_RAM1-I/O4) -> Net-(BIOS_ROM1A-O3)
- BIOS_ROM1 pad 16: Net-(BIOS_RAM1-I/O5) -> Net-(BIOS_ROM1A-O4)
- BIOS_ROM1 pad 17: Net-(BIOS_RAM1-I/O6) -> Net-(BIOS_ROM1A-O5)
- BIOS_ROM1 pad 18: Net-(BIOS_RAM1-I/O7) -> Net-(BIOS_ROM1A-O6)
- BIOS_ROM1 pad 19: Net-(BIOS_RAM1-I/O8) -> Net-(BIOS_ROM1A-O7)
- BIOS_ROM1 pad 2: Net-(BIOS_RAM1-A12) -> Net-(BIOS_ROM1A-A12)
- BIOS_ROM1 pad 21: Net-(BIOS_RAM1-A10) -> Net-(BIOS_ROM1A-A10)
- BIOS_ROM1 pad 23: Net-(BIOS_RAM1-A11) -> Net-(BIOS_ROM1A-A11)
- BIOS_ROM1 pad 24: Net-(BIOS_RAM1-A9) -> Net-(BIOS_ROM1A-A9)
- BIOS_ROM1 pad 25: Net-(BIOS_RAM1-A8) -> Net-(BIOS_ROM1A-A8)
- BIOS_ROM1 pad 26: Net-(BIOS_RAM1-A13) -> Net-(BIOS_ROM1A-A13)
- BIOS_ROM1 pad 27: Net-(BIOS_RAM1-A14) -> Net-(BIOS_ROM1A-A14)
- BIOS_ROM1 pad 3: Net-(BIOS_RAM1-A7) -> Net-(BIOS_ROM1A-A7)
- BIOS_ROM1 pad 4: Net-(BIOS_RAM1-A6) -> Net-(BIOS_ROM1A-A6)
- BIOS_ROM1 pad 5: Net-(BIOS_RAM1-A5) -> Net-(BIOS_ROM1A-A5)
- BIOS_ROM1 pad 6: Net-(BIOS_RAM1-A4) -> Net-(BIOS_ROM1A-A4)
- BIOS_ROM1 pad 7: Net-(BIOS_RAM1-A3) -> Net-(BIOS_ROM1A-A3)
- BIOS_ROM1 pad 8: Net-(BIOS_RAM1-A2) -> Net-(BIOS_ROM1A-A2)
- BIOS_ROM1 pad 9: Net-(BIOS_RAM1-A1) -> Net-(BIOS_ROM1A-A1)
- IC1 pad 1: alu_a_src_5 -> gl_wrt
- IC1 pad 10: Net-(IC179A-1Y) -> (no net)
- IC1 pad 11: /w2 -> clk
- IC1 pad 12: /xbus3 -> Net-(IC1A-5Q)
- IC1 pad 13: Net-(IC179A-2Y) -> /zbus4
- IC1 pad 14: /w3 -> /zbus5
- IC1 pad 15: GND -> Net-(IC1A-6Q)
- IC1 pad 16: (no net) -> Net-(IC1A-7Q)
- IC1 pad 2: /w0 -> Net-(IC1A-1Q)
- IC1 pad 3: Net-(IC170A-1Y) -> /zbus0
- IC1 pad 4: /xbus0 -> /zbus1
- IC1 pad 5: /w1 -> Net-(IC1A-2Q)
- IC1 pad 6: Net-(IC170A-2Y) -> Net-(IC1A-3Q)
- IC1 pad 7: /xbus1 -> /zbus2
- IC1 pad 8: (no net) -> /zbus3
- IC1 pad 9: /xbus2 -> Net-(IC1A-4Q)
- IC100 pad 1: Net-(IC100A-~{A}/B) -> rst
- IC100 pad 10: GND -> (no net)
- IC100 pad 11: GND -> ~{clk}
- IC100 pad 12: unconnected-(IC100A-4Y-Pad12) -> of_in_src_1
- IC100 pad 13: GND -> Net-(IC100A-D5)
- IC100 pad 14: GND -> Net-(IC100A-D6)
- IC100 pad 15: GND -> of_in_src_2
- IC100 pad 16: (no net) -> rd
- IC100 pad 2: GND -> cf_in_src_2
- IC100 pad 3: u_offset_6 -> Net-(IC100A-D1)
- IC100 pad 4: Net-(IC100A-1Y) -> Net-(IC100A-D2)
- IC100 pad 5: GND -> sf_in_src_0
- IC100 pad 6: u_offset_6 -> sf_in_src_1
- IC100 pad 7: Net-(IC100A-2Y) -> Net-(IC100A-D3)
- IC100 pad 8: (no net) -> Net-(IC100A-D4)
- IC100 pad 9: unconnected-(IC100A-3Y-Pad9) -> of_in_src_0
- IC101 pad 1: pch_wrt -> rst
- IC101 pad 11: clk -> ~{clk}
- IC101 pad 12: /pch4 -> dl_wrt
- IC101 pad 13: /zbus4 -> Net-(IC101A-D5)
- IC101 pad 14: /zbus5 -> Net-(IC101A-D6)
- IC101 pad 15: /pch5 -> dh_wrt
- IC101 pad 16: /pch6 -> cl_wrt
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Other:
- board size 1066 x 710 mm -> 1039 x 642 mm

Commit message: kicad
Parts:
- removed IC43, IC46, IC52: 7408N, Package_DIP:DIP-14_W7.62mm
- removed IC86: 7486N, Package_DIP:DIP-14_W7.62mm
- moved IC185 643.3 mm to (714.4, -62.5)
- moved X1 642.1 mm to (737.4, -59.2)
- moved SW2 635.1 mm to (618.4, -60.1)
- moved SW5 620.9 mm to (636.4, -60.5)
- moved IC171 596.1 mm to (645.4, -95.5)
- moved IC175 596.1 mm to (656.2, -95.5)
- moved IC17 585.3 mm to (-372.8, 204.1)
- moved IC19 585.3 mm to (-351.1, 204.1)
- moved IC20 585.3 mm to (-340.2, 204.1)
- moved IC18 585.3 mm to (-361.9, 204.1)
- moved U16 576.6 mm to (655.4, -63.0)
- moved IC23 572.5 mm to (-344.0, 86.5)
- moved IC48 570.9 mm to (-355.0, 132.9)
- moved IC13 551.3 mm to (-329.0, 126.5)
- moved IC115 546.5 mm to (550.0, 104.8)
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Connections:
- IC13 pad 10: (no net) -> /any_interruption
- IC13 pad 11: (no net) -> /mux_a
- IC13 pad 12: (no net) -> typ_1
- IC13 pad 13: (no net) -> Net-(IC13D-I1)
- IC13 pad 4: (no net) -> typ_1
- IC13 pad 5: (no net) -> Net-(IC13B-I1)
- IC13 pad 6: (no net) -> /mux_b
- IC13 pad 8: (no net) -> Net-(IC13C-O)
- IC13 pad 9: (no net) -> Net-(IC13B-I1)
- IC21 pad 8: Net-(IC21D-O) -> Net-(IC13B-I1)
- IC37 pad 1: (no net) -> cond_invert
- IC37 pad 2: (no net) -> /condition
- IC37 pad 3: (no net) -> /final_condition
- IC48 pad 5: Net-(IC46A-O) -> Net-(IC13C-O)
- IC48 pad 6: Net-(IC48B-O) -> Net-(IC13D-I1)
Routing:
- net GND: track 0.00 -> 54.9 mm
- net /u_ad7: track 0.00 -> 48.1 mm
- net /u_ad8: track 0.00 -> 48.0 mm
- net /u_ad13: track 0.00 -> 48.0 mm
- net Net-(IC94A-D4): track 0.00 -> 40.0 mm
- net Net-(IC94A-D7): track 0.00 -> 34.5 mm
- net Net-(IC94A-D2): track 0.00 -> 32.9 mm
- net Net-(IC94A-D1): track 0.00 -> 32.9 mm
- net Net-(IC95A-D2): track 0.00 -> 32.8 mm
- net Net-(IC95A-D1): track 0.00 -> 32.8 mm
- net Net-(IC94A-D3): track 0.00 -> 30.8 mm
- net Net-(IC95A-D3): track 0.00 -> 30.7 mm
- net Net-(IC95A-D4): track 0.00 -> 29.1 mm, vias 0 -> 1
- net Net-(IC95A-D8): track 0.00 -> 26.6 mm
- net Net-(IC95A-D7): track 0.00 -> 26.6 mm
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
Commit message: kicad
Parts:
- moved IC100 667.2 mm to (308.8, 179.4)
- moved IC101 667.2 mm to (310.8, 217.5)
- moved IC102 667.2 mm to (310.2, 255.6)
- moved IC103 667.2 mm to (310.8, 293.8)
- moved IC104 667.2 mm to (353.8, 141.3)
- moved IC105 667.2 mm to (353.8, 179.9)
- moved IC106 667.2 mm to (353.8, 218.6)
- moved IC107 667.2 mm to (353.8, 257.2)
- moved IC108 667.2 mm to (353.8, 295.8)
- moved IC94 667.2 mm to (260.8, 141.9)
- moved IC95 667.2 mm to (260.8, 180.9)
- moved IC96 667.2 mm to (260.8, 219.8)
- moved IC97 667.2 mm to (260.8, 258.8)
- moved IC98 667.2 mm to (260.8, 297.8)
- moved IC99 667.2 mm to (307.8, 141.3)
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Connections:
- IC91 pad 10: (no net) -> GND
- IC91 pad 20: (no net) -> VCC
- IC92 pad 10: (no net) -> GND
- IC92 pad 20: (no net) -> VCC
Routing:
- net GND: track 54.9 -> 309.7 mm, vias 0 -> 4
- net /u_ad12: track 0.00 -> 239.7 mm
- net /u_ad6: track 0.00 -> 103.2 mm, vias 0 -> 2
- net /u_ad3: track 0.00 -> 98.5 mm, vias 0 -> 5
- net /u_ad5: track 0.00 -> 97.6 mm, vias 0 -> 2
- net /u_ad0: track 0.00 -> 70.4 mm, vias 0 -> 4
- net /u_ad7: track 48.1 -> 98.1 mm, vias 0 -> 1
- net /u_ad4: track 0.00 -> 48.9 mm, vias 0 -> 2
- net /u_ad2: track 0.00 -> 48.3 mm, vias 0 -> 2
- net /u_ad1: track 0.00 -> 48.0 mm, vias 0 -> 3
- net /u_ad13: track 48.0 -> 92.6 mm
- net /u_ad9: track 0.00 -> 43.9 mm
- net /u_ad8: track 48.0 -> 91.4 mm, vias 0 -> 4
- net /u_ad11: track 0.00 -> 42.4 mm, vias 0 -> 2
- net /u_ad10: track 0.00 -> 40.5 mm, vias 0 -> 2
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Other:
- board size 1039 x 642 mm -> 1139 x 769 mm

Commit message: kicad
Parts:
- removed the IC28 at (498.6, 164.3)
- removed the IC31 at (520.3, 164.3)
- removed the IC32 at (531.1, 164.3)
- removed the IC33 at (542.0, 164.3)
- removed the IC34 at (552.9, 164.3)
- added IC28: 74151N, Package_DIP:DIP-16_W7.62mm, F.Cu at (1.12, 1.57)
- added IC28: 74151N, Package_DIP:DIP-16_W7.62mm, F.Cu at (329.2, 686.1)
- added IC31: 74253N, Package_DIP:DIP-16_W7.62mm, F.Cu at (349.4, 600.3)
- added IC31: 74253N, Package_DIP:DIP-16_W7.62mm, F.Cu at (12.0, 1.57)
- added IC32: 74253N, Package_DIP:DIP-16_W7.62mm, F.Cu at (22.8, 1.57)
- added IC32: 74253N, Package_DIP:DIP-16_W7.62mm, F.Cu at (349.4, 624.2)
- added IC33: 74253N, Package_DIP:DIP-16_W7.62mm, F.Cu at (33.7, 1.57)
- added IC33: 74253N, Package_DIP:DIP-16_W7.62mm, F.Cu at (349.4, 648.0)
- added IC34: 74253N, Package_DIP:DIP-16_W7.62mm, F.Cu at (349.4, 671.9)
- added IC34: 74253N, Package_DIP:DIP-16_W7.62mm, F.Cu at (44.5, 1.57)
- added IC_10_1: 7410N, Package_DIP:DIP-14_W7.62mm, F.Cu at (1.12, 23.5)
- added IC_10_2: 7410N, Package_DIP:DIP-14_W7.62mm, F.Cu at (689.4, 348.0)
- moved IC45 626.3 mm to (127.4, 325.0)
- moved IC10 615.6 mm to (308.4, 716.2)
- moved IC35 611.0 mm to (189.4, 357.0)
- moved IC177 611.0 mm to (952.5, 568.8)
- moved IC178 611.0 mm to (963.4, 568.8)
- moved IC44 603.1 mm to (127.4, 275.5)
- moved IC16 593.5 mm to (308.2, 667.1)
- moved IC8 591.6 mm to (287.2, 690.7)
- moved IC9 589.7 mm to (308.4, 692.7)
- moved IC7 565.7 mm to (287.2, 667.1)
- moved IC15 563.2 mm to (308.2, 638.7)
- moved IC6 538.2 mm to (287.4, 641.9)
- moved IC75 529.5 mm to (329.4, 555.9)
- moved IC12 529.3 mm to (308.4, 611.8)
- moved IC51 528.5 mm to (329.2, 581.5)
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
Commit message: kicad
Parts:
- removed the IC28 at (1.12, 1.57)
- removed the IC31 at (12.0, 1.57)
- removed the IC32 at (22.8, 1.57)
- removed the IC33 at (33.7, 1.57)
- removed the IC34 at (44.5, 1.57)
- removed the IC_10_1 at (1.12, 23.5)
- added C1: C, Capacitor_THT:C_Disc_D7.5mm_W4.4mm_P5.00mm, F.Cu at (785.0, 242.0)
- added U18: 74LS173, Package_DIP:DIP-16_W7.62mm, F.Cu at (1019.2, 472.1)
- moved IC123 794.2 mm to (68.5, 531.2)
- moved IC124 793.5 mm to (80.0, 531.2)
- moved IC139 783.0 mm to (68.3, 560.9)
- moved IC140 782.4 mm to (79.8, 560.9)
- moved IC141 781.7 mm to (91.3, 560.9)
- moved IC62 778.4 mm to (142.0, 437.4)
- moved IC60 774.6 mm to (124.4, 437.4)
- moved IC58 770.9 mm to (106.8, 437.4)
- moved IC61 770.8 mm to (125.0, 474.0)
- moved IC56 767.1 mm to (89.2, 437.4)
- moved IC59 767.0 mm to (107.3, 474.0)
- moved IC57 763.2 mm to (89.7, 474.0)
- moved IC54 762.9 mm to (72.0, 437.4)
- moved IC109 761.0 mm to (109.7, 590.9)
- moved IC55 759.4 mm to (72.0, 474.0)
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Connections:
- IC171 pad 16: (no net) -> unconnected-(IC171A-VCC-Pad16)
- IC171 pad 8: (no net) -> unconnected-(IC171A-GND-Pad8)
- IC_10_1 pad 10: Net-(IC122A-I1) -> (no net)
- IC_10_1 pad 11: /buffered_mem_io -> (no net)
- IC_10_1 pad 8: Net-(BIOS_ROM1A-~{CE}) -> (no net)
- IC_10_1 pad 9: Net-(IC113A-O) -> (no net)
Other:
- board size 1139 x 769 mm -> 1147 x 796 mm
- board text added: "WBus Multiplexer"

Commit message: kicad
Parts:
- removed IRQ_4_DFF1, IRQ_5_DFF1, IRQ_6_DFF1, IRQ_7_DFF1: 7474N, Package_DIP:DIP-14_W7.62mm
- added U17: 74HC04, Package_DIP:DIP-14_W7.62mm, F.Cu at (591.2, 169.4)
- added U19: 74HC04, Package_DIP:DIP-14_W7.62mm, F.Cu at (474.0, 400.3)
- moved IC159 598.6 mm to (940.3, 554.1)
- moved IC160 598.6 mm to (951.1, 554.1)
- moved IC191 598.6 mm to (940.3, 576.0)
- moved IC1 583.6 mm to (957.5, 584.8)
- moved IC2 583.6 mm to (968.4, 584.8)
- moved IC84 446.3 mm to (889.5, 671.3)
- moved IC85 446.3 mm to (900.4, 671.3)
- moved IC120 411.9 mm to (873.7, 674.7)
- moved IC180 411.9 mm to (928.0, 674.7)
- moved IC117 411.9 mm to (841.1, 674.7)
- moved IC118 411.9 mm to (852.0, 674.7)
- moved IC119 411.9 mm to (862.9, 674.7)
- moved IC179 411.9 mm to (917.1, 674.7)
- moved IC158 399.8 mm to (948.4, 470.3)
- moved IC190 399.8 mm to (948.4, 492.2)
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Connections:
- U18 pad 16: VCC -> unconnected-(U18-VCC-Pad16)
- U18 pad 8: GND -> unconnected-(U18-GND-Pad8)
Other:
- board size 1147 x 796 mm -> 829 x 694 mm
- board text removed: "WBus Multiplexer"
