File: hardware/schematics/kicad/main.kicad_pcb (KiCad board)
At the start: 2 copper layers, 829 x 694 mm, 287 parts, among them IC1 74377N, IC10 74153N, IC100 74273N, IC101 74273N, IC102 74273N, IC103 74273N, IC104 74273N, IC105 74273N, IC106 74273N, IC107 74273N, IC108 74273N, IC109 7427N, IC11 74257N, IC110 74245N, IC111 74257N, IC112 74257N, IC113 7404N, IC114 74377N, IC115 74244N, IC116 74138N, IC117 74244N, IC118 74244N, IC119 74244N, IC12 74257N, IC120 74244N, IC121 7404N, IC122 7420N, IC123 74151N, IC124 74151N, IC125 74151N, IC126 74151N, IC127 74151N, IC128 74151N, IC129 74151N, IC13 7408N, IC130 74151N, IC131 74151N, IC132 74151N, IC133 74151N, IC134 74151N, IC135 74151N, IC136 74151N, IC137 74151N, IC138 74151N, IC139 74151N, IC14 74153N, IC140 74151N, IC141 74151N, IC142 74151N, IC143 74151N, IC144 74151N, IC145 74151N, IC146 74151N, IC147 74151N, IC148 74151N, IC149 74151N, IC15 74257N, IC150 74151N, IC151 74151N, IC152 74151N, IC153 74151N, IC154 74151N, IC155 74257N, IC156 74257N, IC157 74257N, IC158 74257N, IC159 74257N, IC16 74257N, IC160 74257N, IC161 7408N, IC162 7430N, IC163 7404N, IC164 7474N, IC165 7427N, IC166 74153N, IC167 74153N, IC168 74153N, IC169 74153N, IC17 74153N, IC170 7474N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

Commit message: kicad
Parts:
- moved IC84 596.1 mm to (355.0, 407.5)
- moved IC85 590.7 mm to (355.0, 444.5)
- moved IC53 576.8 mm to (337.4, 381.4)
- moved IC1 547.6 mm to (416.4, 501.0)
- moved IC2 542.5 mm to (432.4, 501.0)
- moved IC195 422.1 mm to (548.4, 515.9)
- moved IC194 412.4 mm to (548.4, 462.7)
- moved IC192 397.5 mm to (548.4, 488.7)
- moved IC190 381.2 mm to (567.4, 505.4)
- moved IC180 377.4 mm to (567.6, 562.8)
- moved IC191 375.1 mm to (567.6, 533.8)
- moved IC196 373.2 mm to (567.4, 471.7)
- moved IC197 362.4 mm to (584.4, 433.0)
- moved IC160 348.8 mm to (602.6, 567.8)
- moved IC158 348.0 mm to (603.2, 514.5)
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Other:
- board size 829 x 694 mm -> 1116 x 779 mm
- board text added: "Page Table Block"

Commit message: kicad
Parts:
- removed IC188, IC189: 74279N, Package_DIP:DIP-16_W7.62mm
- removed RN9: R_Pack08, Package_DIP:DIP-16_W7.62mm
- removed SW3: SW_DIP_x08, Package_DIP:DIP-16_W7.62mm
- added S1: 100SP1T1B4M2QE, kicad_models:SW_100SP1T1B4M2QE, F.Cu at (737.7, 578.9)
- added SW11: SW_SPST, kicad_models:SW_100SP1T1B4M2QE, F.Cu at (767.3, 578.9)
- added SW12: SW_SPST, kicad_models:SW_100SP1T1B4M2QE, F.Cu at (708.0, 578.9)
- added SW13: SW_SPST, kicad_models:SW_100SP1T1B4M2QE, F.Cu at (722.8, 578.9)
- added U35: 74HC04, Package_DIP:DIP-14_W7.62mm, F.Cu at (770.6, 636.0)
- SW1: value SW_DIP_x08 -> SW_SPST; footprint Package_DIP:DIP-16_W7.62mm -> kicad_models:SW_100SP1T1B4M2QE
- moved SW4 476.9 mm to (673.7, 604.8)
- moved RN2 402.8 mm to (593.0, 641.5)
- moved RN1 367.5 mm to (654.2, 604.8)
- moved RN8 346.5 mm to (693.2, 604.8)
- moved IC187 339.0 mm to (654.6, 573.8)
- moved IC164 318.9 mm to (732.6, 662.7)
- moved IC170 318.9 mm to (752.2, 662.7)
- moved RN7 315.9 mm to (671.4, 573.8)
- moved IC175 293.8 mm to (752.0, 633.6)
- moved SW10 286.3 mm to (688.2, 573.8)
- moved X1 274.5 mm to (703.2, 642.5)
- moved SW5 236.0 mm to (751.7, 604.8)
- moved SW2 235.2 mm to (732.2, 604.8)
- moved U16 228.6 mm to (712.7, 604.8)
- moved IC185 228.1 mm to (771.2, 604.8)
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Connections:
- RN1 pad 4: /panel_regsel_4 -> panel_regsel_4
- RN1 pad 5: /panel_regsel_3 -> panel_regsel_3
- RN1 pad 6: /panel_regsel_2 -> panel_regsel_2
- RN1 pad 7: /panel_regsel_1 -> panel_regsel_1
- RN1 pad 8: /panel_regsel_0 -> panel_regsel_0
- RN2 pad 1: int_0 -> GND
- RN2 pad 10: VCC -> irq6
- RN2 pad 11: VCC -> irq5
- RN2 pad 12: VCC -> irq4
- RN2 pad 13: VCC -> irq3
- RN2 pad 14: VCC -> irq2
- RN2 pad 15: VCC -> irq1
- RN2 pad 16: VCC -> irq0
- RN2 pad 2: int_1 -> GND
- RN2 pad 3: int_2 -> GND
- RN2 pad 4: int_3 -> GND
- RN2 pad 5: int_4 -> GND
- RN2 pad 6: int_5 -> GND
- RN2 pad 7: int_6 -> GND
- RN2 pad 8: int_7 -> GND
- RN2 pad 9: VCC -> irq7
- RN7 pad 1: Net-(IC189A-R) -> Net-(IC187C-R)
- RN7 pad 2: Net-(IC189A-S1) -> Net-(IC187C-S)
- RN7 pad 3: Net-(IC188A-R) -> Net-(IC187B-R)
- RN7 pad 4: Net-(IC188A-S1) -> Net-(IC187B-S1)
- RN8 pad 1: GND -> Net-(IC164B-D)
- RN8 pad 10: unconnected-(RN8-R7.2-Pad10) -> GND
- RN8 pad 11: Net-(IC187A-R) -> GND
- RN8 pad 12: Net-(IC187A-S1) -> GND
- RN8 pad 13: Net-(IC188A-S1) -> GND
- RN8 pad 14: Net-(IC188A-R) -> GND
- RN8 pad 15: Net-(IC189A-S1) -> GND
- RN8 pad 16: Net-(IC189A-R) -> GND
- RN8 pad 2: GND -> rst
- RN8 pad 3: GND -> unconnected-(RN8-R3.1-Pad3)
- RN8 pad 4: GND -> unconnected-(RN8-R4.1-Pad4)
- RN8 pad 5: GND -> unconnected-(RN8-R5.1-Pad5)
- RN8 pad 6: GND -> unconnected-(RN8-R6.1-Pad6)
- RN8 pad 7: GND -> /stop_clk_req
- RN8 pad 8: GND -> Net-(IC164A-D)
- RN8 pad 9: unconnected-(RN8-R8.2-Pad9) -> GND
- SW1 pad 1: GND -> VCC
- SW1 pad 2: GND -> Net-(IC164B-D)
- SW1 pad 3: GND -> (no net)
- SW10 pad 10: VCC -> GND
- SW10 pad 11: VCC -> GND
- SW10 pad 12: VCC -> GND
- SW10 pad 13: VCC -> GND
- SW10 pad 14: VCC -> GND
- SW10 pad 15: VCC -> GND
- SW10 pad 16: VCC -> GND
- SW10 pad 3: Net-(IC187A-R) -> Net-(IC187A-S1)
- SW10 pad 4: Net-(IC187A-S1) -> Net-(IC187A-R)
- SW10 pad 5: Net-(IC188A-S1) -> Net-(IC187B-S1)
- SW10 pad 6: Net-(IC188A-R) -> Net-(IC187B-R)
- SW10 pad 7: Net-(IC189A-S1) -> Net-(IC187C-S)
- SW10 pad 8: Net-(IC189A-R) -> Net-(IC187C-R)
- SW10 pad 9: VCC -> GND
- SW2 pad 10: Net-(IC121A-I) -> Net-(U18-Cp)
- SW2 pad 11: Net-(IC121A-I) -> Net-(U18-Cp)
- SW2 pad 12: Net-(IC121A-I) -> Net-(U18-Cp)
- SW2 pad 13: Net-(IC121A-I) -> Net-(U18-Cp)
- SW2 pad 14: Net-(IC121A-I) -> Net-(U18-Cp)
- SW2 pad 15: Net-(IC121A-I) -> Net-(U18-Cp)
- SW2 pad 16: Net-(IC121A-I) -> Net-(U18-Cp)
- SW2 pad 9: Net-(IC121A-I) -> Net-(U18-Cp)
- SW4 pad 1: /panel_regsel_0 -> panel_regsel_0
- SW4 pad 2: /panel_regsel_1 -> panel_regsel_1
- SW4 pad 3: /panel_regsel_2 -> panel_regsel_2
- SW4 pad 4: /panel_regsel_3 -> panel_regsel_3
- SW4 pad 5: /panel_regsel_4 -> panel_regsel_4
- U13 pad 30: uart_1_irq -> irq1
- U14 pad 30: uart_0_irq -> irq0
- U18 pad 16: unconnected-(U18-VCC-Pad16) -> VCC
- U18 pad 3: Net-(IC121B-I) -> Net-(U18-Q0)
- U18 pad 7: Net-(IC121A-I) -> Net-(U18-Cp)
- U18 pad 8: unconnected-(U18-GND-Pad8) -> GND

Commit message: kicad
Parts:
- moved IC155 7.31 mm to (677.0, 250.4)
Changed lines of the file:
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@@
   )
   (footprint "Package_DIP:DIP-16_W7.62mm" (layer "F.Cu")
-    (at 684.2 249.125)
+    (at 677 250.38)
     (descr "16-lead though-hole mounted DIP package, row spacing 7.62 mm (300 mils)")
     (tags "THT DIP DIL PDIP 2.54mm 7.62mm 300mil")

Commit message: kicad
Parts:
- removed IC171: 74173N, Package_DIP:DIP-16_W7.62mm
- removed IC199, IC201, IC203, IC205: 74244N, Package_DIP:DIP-20_W7.62mm
- added DIS1: ~, led-displays-obsolete:TIL311, F.Cu at (797.0, 580.5)
- added DIS2: ~, led-displays-obsolete:TIL311, F.Cu at (782.8, 580.5)
- added IC43: 7404N, Package_DIP:DIP-14_W7.62mm, F.Cu at (577.2, 641.4)
- added IC46: 7400N, Package_DIP:DIP-14_W7.62mm, F.Cu at (659.0, 715.4)
- added IC52: 7400N, Package_DIP:DIP-14_W7.62mm, F.Cu at (643.4, 720.0)
- BIOS_ROM1: footprint Package_DIP:DIP-32_W15.24mm -> Package_DIP:DIP-28_W15.24mm
- IC177, IC178: footprint Package_DIP:DIP-28_W7.62mm -> Package_DIP:DIP-28_W15.24mm
- moved IC206 350.4 mm to (924.4, 620.9)
- moved SW9 350.1 mm to (906.0, 577.1)
- moved RN6 335.3 mm to (887.0, 576.8)
- moved SW8 328.5 mm to (906.0, 550.1)
- moved IC204 326.8 mm to (924.4, 589.9)
- moved RN5 310.3 mm to (887.0, 550.0)
- moved SW7 308.1 mm to (906.0, 523.1)
- moved IC202 306.0 mm to (924.4, 558.9)
- moved SW6 289.2 mm to (906.0, 496.1)
- moved IC200 288.8 mm to (924.4, 527.9)
- moved RN4 286.1 mm to (887.0, 523.2)
- moved IC198 275.6 mm to (924.4, 496.9)
- moved RN3 262.9 mm to (887.0, 496.5)
- moved IC157 8.20 mm to (611.4, 488.8)
- moved IC117 8.00 mm to (630.2, 466.1)
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Connections:
- IC111 pad 11: /panel_regsel_2 -> panel_regsel_2
- IC111 pad 14: /panel_regsel_3 -> panel_regsel_3
- IC111 pad 2: /panel_regsel_0 -> panel_regsel_0
- IC111 pad 5: /panel_regsel_1 -> panel_regsel_1
- IC112 pad 2: /panel_regsel_4 -> panel_regsel_4
- IC113 pad 8: Net-(IC113D-O) -> (no net)
- IC113 pad 9: rd -> (no net)
- IC121 pad 1: Net-(IC121A-I) -> (no net)
- IC121 pad 2: Net-(IC121A-O) -> (no net)
- IC121 pad 3: Net-(IC121B-I) -> (no net)
- IC121 pad 4: /clk_crystal -> (no net)
- IC121 pad 5: rst -> (no net)
- IC121 pad 6: ~{rst} -> (no net)
- IC155 pad 12: unconnected-(IC155A-4Y-Pad12) -> display_register3
- IC155 pad 4: unconnected-(IC155A-1Y-Pad4) -> display_register0
- IC155 pad 7: unconnected-(IC155A-2Y-Pad7) -> display_register1
- IC155 pad 9: unconnected-(IC155A-3Y-Pad9) -> display_register2
- IC156 pad 12: unconnected-(IC156A-4Y-Pad12) -> display_register7
- IC156 pad 4: unconnected-(IC156A-1Y-Pad4) -> display_register4
- IC156 pad 7: unconnected-(IC156A-2Y-Pad7) -> display_register5
- IC156 pad 9: unconnected-(IC156A-3Y-Pad9) -> display_register6
- IC163 pad 1: clk -> (no net)
- IC163 pad 2: ~{clk} -> (no net)
- IC170 pad 3: Net-(IC121A-O) -> Net-(IC170A-CLK)
- IC187 pad 10: (no net) -> Net-(IC187B-R)
- IC187 pad 11: (no net) -> Net-(IC187B-S1)
- IC187 pad 12: (no net) -> Net-(IC187B-S1)
- IC187 pad 5: (no net) -> Net-(IC187C-R)
- IC187 pad 6: (no net) -> Net-(IC187C-S)
- IC187 pad 7: (no net) -> panel_wr
- IC187 pad 9: (no net) -> panel_rd
- IC196 pad 2: Net-(IC113D-O) -> Net-(IC196A-A1)
- IC196 pad 4: Net-(IC193D-O) -> Net-(IC196A-A2)
- IC198 pad 11: (no net) -> /panel_address_4
- IC198 pad 13: (no net) -> /panel_address_5
- IC198 pad 15: (no net) -> /panel_address_6
- IC198 pad 17: (no net) -> /panel_address_7
- IC198 pad 19: (no net) -> GND
- IC198 pad 3: (no net) -> address_bus7
- IC198 pad 5: (no net) -> address_bus6
- IC198 pad 7: (no net) -> address_bus5
- IC198 pad 9: (no net) -> address_bus4
- IC200 pad 11: (no net) -> /panel_address_12
- IC200 pad 13: (no net) -> /panel_address_13
- IC200 pad 15: (no net) -> /panel_address_14
- IC200 pad 17: (no net) -> /panel_address_15
- IC200 pad 19: (no net) -> GND
- IC200 pad 3: (no net) -> address_bus15
- IC200 pad 5: (no net) -> address_bus14
- IC200 pad 7: (no net) -> address_bus13
- IC200 pad 9: (no net) -> address_bus12
- IC202 pad 11: (no net) -> /panel_address_20
- IC202 pad 13: (no net) -> /panel_address_21
- IC202 pad 15: (no net) -> GND
- IC202 pad 17: (no net) -> GND
- IC202 pad 19: (no net) -> GND
- IC202 pad 3: (no net) -> unconnected-(IC202B-Y4-Pad3)
- IC202 pad 5: (no net) -> unconnected-(IC202B-Y3-Pad5)
- IC202 pad 7: (no net) -> address_bus21
- IC202 pad 9: (no net) -> address_bus20
- IC204 pad 11: (no net) -> /panel_data_0
- IC204 pad 13: (no net) -> /panel_data_1
- IC204 pad 15: (no net) -> /panel_data_2
- IC204 pad 17: (no net) -> /panel_data_3
- IC204 pad 19: (no net) -> GND
- IC204 pad 3: (no net) -> data_bus3
- IC204 pad 5: (no net) -> data_bus2
- IC204 pad 7: (no net) -> data_bus1
- IC204 pad 9: (no net) -> data_bus0
- IC21 pad 5: mdr_out_en -> (no net)
- IC21 pad 6: Net-(IC21C-O) -> (no net)
- IC42 pad 18: data_bus7 -> unconnected-(IC42A-8D-Pad18)
- IRQ_0_DFF1 pad 10: (no net) -> VCC
- IRQ_0_DFF1 pad 11: (no net) -> irq1
- IRQ_0_DFF1 pad 12: (no net) -> VCC
- IRQ_0_DFF1 pad 13: (no net) -> Net-(IRQ_0_DFF1B-CLR)
- IRQ_0_DFF1 pad 3: uart_0_irq -> irq0
- IRQ_0_DFF1 pad 8: (no net) -> unconnected-(IRQ_0_DFF1B-~{Q}-Pad8)
- IRQ_0_DFF1 pad 9: (no net) -> Net-(IRQ_0_DFF1B-Q)
- IRQ_1_DFF1 pad 1: (no net) -> Net-(IRQ_1_DFF1A-CLR)
- IRQ_1_DFF1 pad 11: uart_1_irq -> irq3
- IRQ_1_DFF1 pad 2: (no net) -> VCC
- IRQ_1_DFF1 pad 3: (no net) -> irq2
- IRQ_1_DFF1 pad 4: (no net) -> VCC
- IRQ_1_DFF1 pad 5: (no net) -> Net-(IRQ_1_DFF1A-Q)
- IRQ_1_DFF1 pad 6: (no net) -> unconnected-(IRQ_1_DFF1A-~{Q}-Pad6)
- IRQ_2_DFF1 pad 10: (no net) -> VCC
- IRQ_2_DFF1 pad 11: (no net) -> irq5
- IRQ_2_DFF1 pad 12: (no net) -> VCC
- IRQ_2_DFF1 pad 13: (no net) -> Net-(IRQ_2_DFF1B-CLR)
- IRQ_2_DFF1 pad 3: int_req_2 -> irq4
- IRQ_2_DFF1 pad 8: (no net) -> unconnected-(IRQ_2_DFF1B-~{Q}-Pad8)
- IRQ_2_DFF1 pad 9: (no net) -> Net-(IRQ_2_DFF1B-Q)
- IRQ_3_DFF1 pad 1: (no net) -> Net-(IRQ_3_DFF1A-CLR)
- IRQ_3_DFF1 pad 11: int_req_3 -> irq7
- IRQ_3_DFF1 pad 2: (no net) -> VCC
- IRQ_3_DFF1 pad 3: (no net) -> irq6
- IRQ_3_DFF1 pad 4: (no net) -> VCC
- IRQ_3_DFF1 pad 5: (no net) -> Net-(IRQ_3_DFF1A-Q)
- IRQ_3_DFF1 pad 6: (no net) -> unconnected-(IRQ_3_DFF1A-~{Q}-Pad6)
- IRQ_AND_1 pad 1: Net-(IRQ_AND_1A-I0) -> /~{clear_all_irqs}
- IRQ_AND_1 pad 10: Net-(IRQ_AND_1C-I1) -> /~{clear_all_irqs}
- IRQ_AND_1 pad 11: Net-(IRQ_3_DFF1B-CLR) -> Net-(IRQ_1_DFF1B-CLR)
- IRQ_AND_1 pad 12: Net-(IRQ_AND_1D-I0) -> /~{clear_all_irqs}
- IRQ_AND_1 pad 2: /~{clear_all_irqs} -> Net-(IRQ_AND_1A-I1)
- IRQ_AND_1 pad 3: Net-(IRQ_4_DFF1A-CLR) -> Net-(IRQ_0_DFF1A-CLR)
- IRQ_AND_1 pad 5: Net-(IRQ_AND_1B-I1) -> /~{clear_all_irqs}
- IRQ_AND_1 pad 6: Net-(IRQ_1_DFF1B-CLR) -> Net-(IRQ_0_DFF1B-CLR)
- IRQ_AND_1 pad 8: Net-(IRQ_2_DFF1A-CLR) -> Net-(IRQ_1_DFF1A-CLR)
- IRQ_AND_2 pad 11: Net-(IRQ_7_DFF1B-CLR) -> Net-(IRQ_3_DFF1B-CLR)
- IRQ_AND_2 pad 12: Net-(IRQ_AND_2D-I0) -> /~{clear_all_irqs}
- IRQ_AND_2 pad 2: Net-(IRQ_AND_2A-I1) -> /~{clear_all_irqs}
- IRQ_AND_2 pad 3: Net-(IRQ_0_DFF1A-CLR) -> Net-(IRQ_2_DFF1A-CLR)
- IRQ_AND_2 pad 4: Net-(IRQ_AND_2B-I0) -> /~{clear_all_irqs}
- IRQ_AND_2 pad 6: Net-(IRQ_5_DFF1B-CLR) -> Net-(IRQ_2_DFF1B-CLR)
- IRQ_AND_2 pad 8: Net-(IRQ_6_DFF1A-CLR) -> Net-(IRQ_3_DFF1A-CLR)
- IRQ_AND_2 pad 9: Net-(IRQ_AND_2C-I0) -> /~{clear_all_irqs}
- IRQ_ENCODER1 pad 1: Net-(IC207D-O) -> Net-(IC46D-O)
- IRQ_ENCODER1 pad 10: Net-(IC208D-O) -> Net-(IC52D-O)
- IRQ_ENCODER1 pad 11: Net-(IC208C-O) -> Net-(IC52C-O)
- IRQ_ENCODER1 pad 12: Net-(IC208B-O) -> Net-(IC52B-O)
- IRQ_ENCODER1 pad 13: Net-(IC208A-O) -> Net-(IC52A-O)
- IRQ_ENCODER1 pad 2: Net-(IC207C-O) -> Net-(IC46C-O)
- IRQ_ENCODER1 pad 3: Net-(IC207B-O) -> Net-(IC46B-O)
- IRQ_ENCODER1 pad 4: Net-(IC207A-O) -> Net-(IC46A-O)
- IRQ_RST_DECODER1 pad 10: Net-(IRQ_AND_2B-I0) -> /~{clear_all_irqs}
- IRQ_RST_DECODER1 pad 11: Net-(IRQ_AND_1A-I0) -> /~{clear_all_irqs}
- IRQ_RST_DECODER1 pad 12: Net-(IRQ_AND_1D-I0) -> /~{clear_all_irqs}
- IRQ_RST_DECODER1 pad 13: Net-(IRQ_AND_1C-I1) -> /~{clear_all_irqs}
- IRQ_RST_DECODER1 pad 14: Net-(IRQ_AND_1B-I1) -> /~{clear_all_irqs}
- IRQ_RST_DECODER1 pad 15: Net-(IRQ_AND_2A-I1) -> Net-(IRQ_AND_1A-I1)
- IRQ_RST_DECODER1 pad 7: Net-(IRQ_AND_2D-I0) -> /~{clear_all_irqs}
- IRQ_RST_DECODER1 pad 9: Net-(IRQ_AND_2C-I0) -> /~{clear_all_irqs}
- IRQ_STATUS_1 pad 13: Net-(IRQ_4_DFF1A-Q) -> Net-(IRQ_2_DFF1A-Q)
- IRQ_STATUS_1 pad 14: Net-(IRQ_5_DFF1B-Q) -> Net-(IRQ_2_DFF1B-Q)
- IRQ_STATUS_1 pad 17: Net-(IRQ_6_DFF1A-Q) -> Net-(IRQ_3_DFF1A-Q)
- IRQ_STATUS_1 pad 18: Net-(IRQ_7_DFF1B-Q) -> Net-(IRQ_3_DFF1B-Q)
- IRQ_STATUS_1 pad 4: Net-(IRQ_1_DFF1B-Q) -> Net-(IRQ_0_DFF1B-Q)
- IRQ_STATUS_1 pad 7: Net-(IRQ_2_DFF1A-Q) -> Net-(IRQ_1_DFF1A-Q)
- IRQ_STATUS_1 pad 8: Net-(IRQ_3_DFF1B-Q) -> Net-(IRQ_1_DFF1B-Q)
- MDR_OUT_MUX_1 pad 15: Net-(IC21C-O) -> Net-(MDR_OUT_MUX_1A-G)
- MDR_OUT_MUX_2 pad 15: Net-(IC21C-O) -> Net-(MDR_OUT_MUX_1A-G)
