File: hardware/schematics/kicad_wirewrap/main.kicad_sch (KiCad schematic)
At the start: 284 parts, among them IC1 74377N, IC10 74153N, IC100 74273N, IC101 74273N, IC102 74273N, IC103 74273N, IC104 74273N, IC105 74273N, IC106 74273N, IC107 74273N, IC108 74273N, IC109 7427N, IC11 74257N, IC110 74245N, IC111 74257N, IC112 74257N, IC113 7404N, IC114 74377N, IC115 74244N, IC116 74138N, IC117 74244N, IC118 74244N, IC119 74244N, IC12 74257N, IC120 74244N, IC121 7404N, IC122 7420N, IC123 74151N, IC124 74151N, IC125 74151N, IC126 74151N, IC127 74151N, IC128 74151N, IC129 74151N, IC13 7408N, IC130 74151N, IC131 74151N, IC132 74151N, IC133 74151N, IC134 74151N, IC135 74151N, IC136 74151N, IC137 74151N, IC138 74151N, IC139 74151N, IC14 74153N, IC140 74151N, IC141 74151N, IC142 74151N, IC143 74151N, IC144 74151N, IC145 74151N, IC146 74151N, IC147 74151N, IC148 74151N, IC149 74151N, IC15 74257N, IC150 74151N, IC151 74151N, IC152 74151N, IC153 74151N, IC154 74151N, IC155 74257N, IC156 74257N, IC157 74257N, IC158 74257N, IC159 74257N, IC16 74257N, IC160 74257N, IC161 7408N, IC162 7430N, IC163 7404N, IC164 7474N, IC165 7427N, IC166 74153N, IC167 74153N, IC168 74153N, IC169 74153N, IC17 74153N, IC170 7474N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

Commit message: kicad
Parts:
- removed IC43: 7404N, main:DIL14, symbol main-eagle-import:7404N
- removed IC46, IC52: 7400N, main:DIL14, symbol main-eagle-import:7400N
- added IC193: 7404N, main:DIL14, symbol main-eagle-import:7404N
- added IC207, IC208: 7400N, main:DIL14, symbol main-eagle-import:7400N
- added SW3: SW_DIP_x08, Package_DIP:DIP-16_W7.62mm, symbol Switch:SW_DIP_x08
Connections:
- net GND: now also SW3.1, SW3.2, SW3.3, SW3.4, SW3.5, SW3.6, SW3.7, SW3.8; no longer RN2.1 (R1.1), RN2.2 (R2.1), RN2.3 (R3.1), RN2.4 (R4.1), RN2.5 (R5.1), RN2.6 (R6.1), RN2.7 (R7.1), RN2.8 (R8.1)
- net VCC: now also RN2.10 (R7.2), RN2.11 (R6.2), RN2.12 (R5.2), RN2.13 (R4.2), RN2.14 (R3.2), RN2.15 (R2.2), RN2.16 (R1.2), RN2.9 (R8.2)
- net clear_all_irqs: now also IC193.1 (I)
- net int_status_0: now also IC207.2 (I1)
- net int_status_1: now also IC207.5 (I1)
- net int_status_2: now also IC207.10 (I1)
- net int_status_3: now also IC207.13 (I1)
- net int_status_4: now also IC208.2 (I1)
- net int_status_5: now also IC208.5 (I1)
- net int_status_6: now also IC208.10 (I1)
- net int_status_7: now also IC208.13 (I1)
- net irq0: now also RN2.1 (R1.1), SW3.16; no longer RN2.16 (R1.2)
- net irq1: now also RN2.2 (R2.1), SW3.15; no longer RN2.15 (R2.2)
- net irq2: now also RN2.3 (R3.1), SW3.14; no longer RN2.14 (R3.2)
- net irq3: now also RN2.4 (R4.1), SW3.13; no longer RN2.13 (R4.2)
- net irq4: now also RN2.5 (R5.1), SW3.12; no longer RN2.12 (R5.2)
- net irq5: now also RN2.6 (R6.1), SW3.11; no longer RN2.11 (R6.2)
- net irq6: now also RN2.7 (R7.1), SW3.10; no longer RN2.10 (R7.2)
- net irq7: now also RN2.8 (R8.1), SW3.9; no longer RN2.9 (R8.2)
- net irq_masks0: now also IC207.1 (I0)
- net irq_masks1: now also IC207.4 (I0)
- net irq_masks2: now also IC207.9 (I0)
- net irq_masks3: now also IC207.12 (I0)
- net irq_masks4: now also IC208.1 (I0)
- net irq_masks5: now also IC208.4 (I0)
- net irq_masks6: now also IC208.9 (I0)
- net irq_masks7: now also IC208.12 (I0)
- net ~{clear_all_irqs}: now also IC193.2 (O)
- net at IRQ_ENCODER1.10 (0): now also IC208.11 (O)
- net at IRQ_ENCODER1.11 (1): now also IC208.8 (O)
- net at IRQ_ENCODER1.1 (4): now also IC207.11 (O)
- net at IRQ_ENCODER1.12 (2): now also IC208.6 (O)
- net at IRQ_ENCODER1.13 (3): now also IC208.3 (O)
- net at IRQ_ENCODER1.2 (5): now also IC207.8 (O)
- net at IRQ_ENCODER1.3 (6): now also IC207.6 (O)
- net at IRQ_ENCODER1.4 (7): now also IC207.3 (O)
Other:
- moved on the sheet: U1, U10, U11, U12, U13, U14, U2, U3, U4, U5, U6, U7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
